File: 02_Schaltplan/KiCad/Schaltplan/Constant-Current-Logic.kicad_sch (KiCad schematic)
At the start: 42 parts, among them Q1 SI2318, U17 LMV321AUIDBVR, U18 LMV358MM, U19 INA826AIDRGT, U20 74HC595, U21 74HC595, U22 74AHC2G08

Commit message: ADD
-Dokumentation erweitert
-Schaltplan Fußbeschriftungen
Parts:
- U22: BMK-Nr - -> 06-0948-1
Other:
- company: (none) -> BMK Group
- title: (none) -> Kabeltester
Changed lines of the file:
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@@
 (kicad_sch (version 20210126) (generator eeschema)
   (paper "A3")
+  (title_block
+    (title "Kabeltester")
+    (company "BMK Group")
+    (comment 1 "Erstellt: Maximilian Hoffmann")
+    (comment 2 "Geprüft: Robert Schulz")
+  )
   (junction (at 73.025 242.57) (diameter 1.016) (color 0 0 0 0))
   (junction (at 73.025 265.43) (diameter 1.016) (color 0 0 0 0))
@@
       (effects (font (size 1.27 1.27)) hide)
     )
-    (property "BMK-Nr" "-" (id 4) (at 260.35 269.875 0)
+    (property "BMK-Nr" "06-0948-1" (id 4) (at 260.35 269.875 0)
       (effects (font (size 1.27 1.27)) hide)
     )
@@
       (effects (font (size 1.27 1.27)) hide)
     )
-    (property "BMK-Nr" "-" (id 4) (at 256.54 125.095 0)
+    (property "BMK-Nr" "06-0948-1" (id 4) (at 256.54 125.095 0)
       (effects (font (size 1.27 1.27)) hide)
     )
@@
       (effects (font (size 1.27 1.27)) hide)
     )
-    (property "BMK-Nr" "-" (id 4) (at 275.59 131.445 0)
-      (effects (font (size 1.27 1.27)) hide)
-    )
+    (property "BMK-Nr" "06-0948-1" (id 4) (at 275.59 131.445 0)
+      (effects (font (size 1.27 1.27)) hide)
+    )
