File: 02_Schaltplan/KiCad/Schaltplan/Constant-Current-Logic.kicad_sch (KiCad schematic)
At the start: 40 parts, among them Q1 SI2318, U17 LMV321AUIDBVR, U18 LMV358MM, U19 INA826AIDRGT, U20 74HC595, U21 74HC595, U22 74AHC2G08

Commit message: Doku
Schaltplan
-Versorgung
-Taktgeber
Parts:
- removed L2: L, Inductor_SMD:L_TDK_NLV32_3.2x2.5mm, symbol Device:L
- added C?: 100nF, Capacitor_SMD:C_0603_1608Metric_Pad1.08x0.95mm_HandSolder, symbol Device:C
- added R22: 10k, Resistor_SMD:R_0603_1608Metric_Pad0.98x0.95mm_HandSolder, symbol Device:R
- added U9: 74AHC1G14, Package_TO_SOT_SMD:SOT-353_SC-70-5_Handsoldering, symbol Kabeltester:74AHC1G14
- R92: value 0R -> 22R
Connections:
- net +5V: now also C?.1, U9.5 (VCC)
- net GND: now also C?.2, U9.3 (GND)
- net SYSTEM_TACK_2: now also U9.2; no longer U22.2 (1B)
- net at C22.1, TP3.1, U17.3 (-): now also R22.2; no longer U19.7
- new net: U22.2 (1B), U9.4
- new net: R22.1, U19.7
Other:
- moved on the sheet: C22, JP1, JP2, R92, TP3, TP36, TP37, TP6, TP7, U20A, U21A, U22A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

Commit message: ADD
Parts:
- gave numbers to parts that had none: 1
Changed lines of the file:
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@@
   (symbol (lib_id "power:+5V") (at 225.425 242.57 0) (unit 1)
     (in_bom yes) (on_board yes)
-    (property "Reference" "#PWR?" (id 0) (at 225.425 246.38 0)
+    (property "Reference" "#PWR0107" (id 0) (at 225.425 246.38 0)
       (effects (font (size 1.27 1.27)) hide)
     )
@@
   (symbol (lib_id "power:GND") (at 225.425 265.43 0) (unit 1)
     (in_bom yes) (on_board yes)
-    (property "Reference" "#PWR?" (id 0) (at 225.425 271.78 0)
+    (property "Reference" "#PWR0108" (id 0) (at 225.425 271.78 0)
       (effects (font (size 1.27 1.27)) hide)
     )
@@
   (symbol (lib_name "Device:C_8") (lib_id "Device:C") (at 234.95 254.635 0) (unit 1)
     (in_bom yes) (on_board yes)
-    (property "Reference" "C?" (id 0) (at 229.6161 252.2156 0)
-      (effects (font (size 1.27 1.27)) (justify left))
-    )
+    (property "Reference" "C26" (id 0) (at 229.6161 252.2156 0)
+      (effects (font (size 1.27 1.27)) (justify left))
+    )

Commit message: Änderungen
Connections:
- net SYSTEM_TACKT_SR_INV renamed SYSTEM_TAKT_SR_INV
- net SYSTEM_TACK_2 renamed SYSTEM_TAKT_2
Changed lines of the file:
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@@
     )
   )
-  (global_label "SYSTEM_TACK_2" (shape input) (at 242.57 112.395 180)
+  (global_label "SYSTEM_TAKT_2" (shape input) (at 242.57 112.395 180)
     (effects (font (size 1.27 1.27)) (justify right))
     (property "Intersheet References" "${INTERSHEET_REFS}" (id 0) (at 223.8162 112.3156 0)
@@
     )
   )
-  (global_label "SYSTEM_TACKT_SR_INV" (shape input) (at 259.08 106.045 180)
+  (global_label "SYSTEM_TAKT_SR_INV" (shape input) (at 259.08 106.045 180)
     (effects (font (size 1.27 1.27)) (justify right))
     (property "Intersheet References" "${INTERSHEET_REFS}" (id 0) (at 234.0972 105.9656 0)

Commit message: ADD
Parts:
- R87: value 1k -> 36k
- R88: value 1k -> 16k
- R90: value 0R -> 8,2k
- R91: value 0R -> 43k
- RV2, RV3: value 20k -> 2k
Other:
- note added: "Taktpegel-Anpassung & Anzeigen-Logik"
- note removed: "Taktpegel-Anpassung & Anzeigen-Logic"
Changed lines of the file:
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@@
     (effects (font (size 5 5) (thickness 1) bold) (justify right bottom))
   )
-  (text "Taktpegel-Anpassung & Anzeigen-Logic\n\n \n" (at 295.91 64.135 180)
+  (text "Taktpegel-Anpassung & Anzeigen-Logik\n\n\n \n" (at 295.91 64.135 180)
     (effects (font (size 2 2) (thickness 0.4) bold) (justify right bottom))
   )
@@
       (effects (font (size 1.27 1.27)) (justify left))
     )
-    (property "Value" "1k" (id 1) (at 74.422 95.371 0)
+    (property "Value" "36k" (id 1) (at 74.422 95.371 0)
       (effects (font (size 1.27 1.27)) (justify left))
     )
@@
       (effects (font (size 1.27 1.27)) (justify left))
     )
-    (property "Value" "1k" (id 1) (at 74.422 115.691 0)
+    (property "Value" "16k" (id 1) (at 74.422 115.691 0)
       (effects (font (size 1.27 1.27)) (justify left))
     )
@@
       (effects (font (size 1.27 1.27)) (justify left))
     )
-    (property "Value" "0R" (id 1) (at 134.747 170.936 0)
+    (property "Value" "8,2k" (id 1) (at 134.747 170.936 0)
       (effects (font (size 1.27 1.27)) (justify left))
     )
@@
       (effects (font (size 1.27 1.27)) (justify left))
     )
-    (property "Value" "0R" (id 1) (at 134.747 193.161 0)
+    (property "Value" "43k" (id 1) (at 134.747 193.161 0)
       (effects (font (size 1.27 1.27)) (justify left))
     )
@@
       (effects (font (size 1.27 1.27)) (justify right))
     )
-    (property "Value" "20k" (id 1) (at 74.295 106.68 0)
+    (property "Value" "2k" (id 1) (at 74.295 106.68 0)
       (effects (font (size 1.27 1.27)) (justify right))
     )
@@
       (effects (font (size 1.27 1.27)) (justify right))
     )
-    (property "Value" "20k" (id 1) (at 134.62 182.88 0)
+    (property "Value" "2k" (id 1) (at 134.62 182.88 0)
       (effects (font (size 1.27 1.27)) (justify right))
     )

Commit message: ADD
Connections:
- net +5V: no longer C21.1, U19.8 (+VS)
- new net +9V: C21.1, U19.8 (+VS)
Other:
- note added: "Fehler 3"
- note added: "Fehler 4"
- note added: "Fehler 5"
Changed lines of the file:
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@@
     (stroke (width 1) (type solid) (color 255 0 0 1))
+  )
+  (polyline (pts (xy 95.25 234.95) (xy 95.25 243.205))
+    (stroke (width 0.3) (type dash_dot) (color 0 0 255 1))
+  )
+  (polyline (pts (xy 95.25 234.95) (xy 102.235 234.95))
+    (stroke (width 0.3) (type dash_dot) (color 0 0 255 1))
+  )
+  (polyline (pts (xy 102.235 234.95) (xy 102.235 243.205))
+    (stroke (width 0.3) (type dash_dot) (color 0 0 255 1))
+  )
+  (polyline (pts (xy 102.235 243.205) (xy 95.25 243.205))
+    (stroke (width 0.3) (type dash_dot) (color 0 0 255 1))
+  )
+  (polyline (pts (xy 103.505 238.125) (xy 106.045 238.125))
+    (stroke (width 0.3) (type solid) (color 0 0 255 1))
+  )
+  (polyline (pts (xy 104.14 235.585) (xy 103.505 238.125))
+    (stroke (width 0.3) (type solid) (color 0 0 255 1))
+  )
+  (polyline (pts (xy 109.22 233.68) (xy 103.505 238.125))
+    (stroke (width 0.3) (type solid) (color 0 0 255 1))
+  )
+  (polyline (pts (xy 116.205 73.025) (xy 116.205 80.01))
+    (stroke (width 0.3) (type dash_dot) (color 0 0 255 1))
+  )
+  (polyline (pts (xy 116.205 73.025) (xy 124.46 73.025))
+    (stroke (width 0.3) (type dash_dot) (color 0 0 255 1))
+  )
+  (polyline (pts (xy 116.205 80.01) (xy 124.46 80.01))
+    (stroke (width 0.3) (type dash_dot) (color 0 0 255 1))
+  )
+  (polyline (pts (xy 124.46 72.39) (xy 127 72.39))
+    (stroke (width 0.3) (type solid) (color 0 0 255 1))
+  )
+  (polyline (pts (xy 124.46 80.01) (xy 124.46 73.025))
+    (stroke (width 0.3) (type dash_dot) (color 0 0 255 1))
+  )
+  (polyline (pts (xy 125.095 69.85) (xy 124.46 72.39))
+    (stroke (width 0.3) (type solid) (color 0 0 255 1))
+  )
+  (polyline (pts (xy 130.175 67.945) (xy 124.46 72.39))
+    (stroke (width 0.3) (type solid) (color 0 0 255 1))
   )
   (polyline (pts (xy 203.2 50.8) (xy 203.2 133.35))
@@
     (stroke (width 1) (type solid) (color 0 0 255 1))
   )
+  (polyline (pts (xy 230.505 106.68) (xy 239.395 109.855))
+    (stroke (width 0.3) (type solid) (color 0 0 255 1))
+  )
+  (polyline (pts (xy 238.76 107.95) (xy 239.395 109.855))
+    (stroke (width 0.3) (type solid) (color 0 0 255 1))
+  )
+  (polyline (pts (xy 239.395 109.855) (xy 237.49 110.49))
+    (stroke (width 0.3) (type solid) (color 0 0 255 1))
+  )
+  (polyline (pts (xy 242.57 107.95) (xy 243.84 107.95))
+    (stroke (width 0.3) (type dash_dot) (color 0 0 255 1))
+  )
+  (polyline (pts (xy 242.57 116.205) (xy 242.57 107.95))
+    (stroke (width 0.3) (type dash_dot) (color 0 0 255 1))
+  )
+  (polyline (pts (xy 243.84 107.95) (xy 254.635 107.95))
+    (stroke (width 0.3) (type dash_dot) (color 0 0 255 1))
+  )
   (polyline (pts (xy 247.65 273.05) (xy 247.65 228.6))
     (stroke (width 1) (type solid) (color 255 0 0 1))
   )
+  (polyline (pts (xy 254.635 107.95) (xy 254.635 116.205))
+    (stroke (width 0.3) (type dash_dot) (color 0 0 255 1))
+  )
+  (polyline (pts (xy 254.635 116.205) (xy 242.57 116.205))
+    (stroke (width 0.3) (type dash_dot) (color 0 0 255 1))
+  )
   (polyline (pts (xy 400.05 222.25) (xy 400.05 50.8))
     (stroke (width 1) (type solid) (color 0 0 255 1))
@@
     (effects (font (size 2 2) (thickness 0.4) bold) (justify right bottom))
   )
+  (text "Fehler 4\n" (at 104.775 233.68 0)
+    (effects (font (size 1.27 1.27) (thickness 0.254) bold) (justify left bottom))
+  )
   (text "Auswertung Konstantstromquelle\n" (at 118.745 146.685 180)
     (effects (font (size 2 2) (thickness 0.4) bold) (justify right bottom))
   )
+  (text "Fehler 3\n" (at 125.73 67.945 0)
+    (effects (font (size 1.27 1.27) (thickness 0.254) bold) (justify left bottom))
+  )
+  (text "Fehler 5\n" (at 220.98 107.95 0)
+    (effects (font (size 1.27 1.27) (thickness 0.254) bold) (justify left bottom))
+  )
   (text "CONSTANT-CURRENT-LOGIC\n" (at 274.955 27.305 180)
     (effects (font (size 5 5) (thickness 1) bold) (justify right bottom))
   )
-  (text "Taktpegel-Anpassung & Anzeigen-Logik\n\n\n \n" (at 295.91 64.135 180)
+  (text "Taktpegel-Anpassung & Anzeigen-Logik\n\n\n \n" (at 278.13 69.215 180)
     (effects (font (size 2 2) (thickness 0.4) bold) (justify right bottom))
   )
@@
     (pin "1")
   )
-  (symbol (lib_id "power:+5V") (at 98.425 242.57 0) (unit 1)
-    (in_bom yes) (on_board yes)
-    (property "Reference" "#PWR054" (id 0) (at 98.425 246.38 0)
-      (effects (font (size 1.27 1.27)) hide)
-    )
-    (property "Value" "+5V" (id 1) (at 98.7933 238.2456 0))
+  (symbol (lib_id "power:+9V") (at 98.425 242.57 0) (unit 1)
+    (in_bom yes) (on_board yes)
+    (property "Reference" "#PWR?" (id 0) (at 98.425 246.38 0)
+      (effects (font (size 1.27 1.27)) hide)
+    )
+    (property "Value" "+9V" (id 1) (at 99.06 236.855 0))
     (property "Footprint" "" (id 2) (at 98.425 242.57 0)
       (effects (font (size 1.27 1.27)) hide)
@@
   (symbol (lib_name "Kabeltester:INA826AIDRGT_1") (lib_id "Kabeltester:INA826AIDRGT") (at 98.425 254 0) (mirror y) (unit 2)
     (in_bom yes) (on_board yes)
-    (property "Reference" "U19" (id 0) (at 95.25 243.5668 0))
+    (property "Reference" "U19" (id 0) (at 92.075 244.8368 0))
     (property "Value" "INA826AIDRGT" (id 1) (at 93.98 254.1205 90))
     (property "Footprint" "Package_DFN_QFN:DFN-8-1EP_2x2mm_P0.5mm_EP0.6x1.2mm" (id 2) (at 98.425 236.22 0)

Commit message: ADD
Parts:
- U17: Stromaufnahme (none) -> 70uA
- U18: Stromaufnahme (none) -> 130uA
- U19: Stromaufnahme (none) -> 200uA
- U20, U21: Stromaufnahme (none) -> 8uA
- U22, U9: Stromaufnahme (none) -> 1uA
Other:
- note added: "Fehler 6"
- moved on the sheet: C20, C21, C22, C23, C24, C25, C26, C50, C51, JP1, JP2, Q1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

Commit message: Changes
Parts:
- U17: Mouser 595-LMV321AUIDBVR -> (none)
- U18: Mouser 926-LMV358MMX/NOPB -> (none)
- U19: Mouser 595-INA826AIDGK -> (none)
- U20, U21: Mouser 595-CD74HC595M96 -> (none)
Changed lines of the file:
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@@
-    (stroke (width 0) (type solid) (color 0 0 0 0))
-  )
-  (wire (pts (xy 234.95 114.3) (xy 254 114.3))
     (stroke (width 0) (type solid) (color 0 0 0 0))
   )
@@
     )
   )
-  (global_label "SYSTEM_STATUS_SR" (shape input) (at 234.95 114.3 180)
+  (global_label "SYSTEM_STATUS_SR" (shape input) (at 254 114.3 180)
     (effects (font (size 1.27 1.27)) (justify right))
-    (property "Intersheet References" "${INTERSHEET_REFS}" (id 0) (at 212.7491 114.2206 0)
+    (property "Intersheet References" "${INTERSHEET_REFS}" (id 0) (at 231.7991 114.2206 0)
       (effects (font (size 1.27 1.27)) (justify right) hide)
     )
@@
   (symbol (lib_id "Kabeltester:74AHC1G14") (at 223.52 107.95 0) (unit 1)
     (in_bom yes) (on_board yes)
-    (property "Reference" "U9" (id 0) (at 225.425 104.775 0))
-    (property "Value" "74AHC1G14" (id 1) (at 224.155 102.235 0)
-      (effects (font (size 1.27 1.27)) hide)
+    (property "Reference" "U9" (id 0) (at 224.155 114.935 0))
+    (property "Value" "74AHC1G14" (id 1) (at 224.155 113.03 0)
+      (effects (font (size 1.27 1.27) bold))
     )
     (property "Footprint" "Package_TO_SOT_SMD:SOT-353_SC-70-5_Handsoldering" (id 2) (at 238.125 133.35 0)
@@
   (symbol (lib_id "Transistor_FET:BSS123") (at 144.78 98.425 0) (unit 1)
     (in_bom yes) (on_board yes)
-    (property "Reference" "Q1" (id 0) (at 151.13 96.52 0)
-      (effects (font (size 1.27 1.27)) (justify left))
-    )
-    (property "Value" "SI2318" (id 1) (at 151.13 99.06 0)
-      (effects (font (size 1.27 1.27)) (justify left))
+    (property "Reference" "Q1" (id 0) (at 150.495 99.06 0)
+      (effects (font (size 1.27 1.27)) (justify left))
+    )
+    (property "Value" "SI2318" (id 1) (at 150.495 97.155 0)
+      (effects (font (size 1.27 1.27) bold) (justify left))
     )
     (property "Footprint" "Package_TO_SOT_SMD:SOT-23" (id 2) (at 149.86 100.33 0)
@@
       (effects (font (size 1.27 1.27)) hide)
     )
-    (property "Mouser" "595-INA826AIDGK" (id 4) (at 74.295 249.555 0)
-      (effects (font (size 1.27 1.27)) hide)
-    )
     (property "Stromaufnahme" "200uA" (id 5) (at 74.295 249.555 0)
       (effects (font (size 1.27 1.27)) hide)
@@
       (effects (font (size 1.27 1.27)) hide)
     )
-    (property "Mouser" "926-LMV358MMX/NOPB" (id 4) (at 99.695 249.555 0)
-      (effects (font (size 1.27 1.27)) hide)
-    )
     (property "Stromaufnahme" "130uA" (id 5) (at 99.695 249.555 0)
       (effects (font (size 1.27 1.27)) hide)
@@
       (effects (font (size 1.27 1.27)) hide)
     )
-    (property "Mouser" "595-CD74HC595M96" (id 4) (at 125.095 249.555 0)
-      (effects (font (size 1.27 1.27)) hide)
-    )
     (property "Stromaufnahme" "8uA" (id 5) (at 125.095 249.555 0)
       (effects (font (size 1.27 1.27)) hide)
@@
       (effects (font (size 1.27 1.27)) hide)
     )
-    (property "Mouser" "595-CD74HC595M96" (id 4) (at 150.495 249.555 0)
-      (effects (font (size 1.27 1.27)) hide)
-    )
     (property "Stromaufnahme" "8uA" (id 5) (at 150.495 249.555 0)
       (effects (font (size 1.27 1.27)) hide)
@@
       (effects (font (size 1.27 1.27)) hide)
     )
-    (property "Mouser" "595-LMV321AUIDBVR" (id 4) (at 48.895 249.555 0)
-      (effects (font (size 1.27 1.27)) hide)
-    )
     (property "Stromaufnahme" "70uA" (id 5) (at 48.895 249.555 0)
       (effects (font (size 1.27 1.27)) hide)
@@
   (symbol (lib_name "Kabeltester:LMV358MM_2") (lib_id "Kabeltester:LMV358MM") (at 71.12 172.085 0) (unit 1)
     (in_bom yes) (on_board yes)
-    (property "Reference" "U18" (id 0) (at 72.39 166.6048 0))
-    (property "Value" "LMV358MM" (id 1) (at 66.04 172.713 90)
-      (effects (font (size 1.27 1.27)) hide)
+    (property "Reference" "U18" (id 0) (at 74.93 165.3348 0))
+    (property "Value" "LMV358MM" (id 1) (at 74.93 166.998 0)
+      (effects (font (size 1.27 1.27) bold))
     )
     (property "Footprint" "Package_SO:SOIC-8_3.9x4.9mm_P1.27mm" (id 2) (at 71.12 171.45 0)
@@
       (effects (font (size 1.27 1.27)) hide)
     )
-    (property "Mouser" "926-LMV358MMX/NOPB" (id 4) (at 71.12 172.085 0)
-      (effects (font (size 1.27 1.27)) hide)
-    )
     (property "Stromaufnahme" "130uA" (id 5) (at 71.12 172.085 0)
       (effects (font (size 1.27 1.27)) hide)
@@
   (symbol (lib_id "Kabeltester:LMV321AUIDBVR") (at 80.645 98.425 0) (mirror x) (unit 1)
     (in_bom yes) (on_board yes)
-    (property "Reference" "U17" (id 0) (at 80.3911 102.7494 0)
-      (effects (font (size 1.27 1.27)) (justify left))
-    )
-    (property "Value" "LMV321AUIDBVR" (id 1) (at 75.311 91.561 0)
-      (effects (font (size 1.27 1.27)) (justify left) hide)
+    (property "Reference" "U17" (id 0) (at 78.4861 105.2894 0)
+      (effects (font (size 1.27 1.27)) (justify left))
+    )
+    (property "Value" "LMV321AUIDBVR" (id 1) (at 78.486 103.626 0)
+      (effects (font (size 1.27 1.27) bold) (justify left))
     )
     (property "Footprint" "Package_TO_SOT_SMD:SOT-23-5_HandSoldering" (id 2) (at 80.645 98.425 0)
@@
     )
     (property "BMK-Nr" "11-1946" (id 4) (at 80.645 98.425 0)
-      (effects (font (size 1.27 1.27)) hide)
-    )
-    (property "Mouser" "595-LMV321AUIDBVR" (id 4) (at 80.645 98.425 0)
       (effects (font (size 1.27 1.27)) hide)
     )
@@
   (symbol (lib_id "Kabeltester:LMV358MM") (at 143.51 174.625 0) (unit 2)
     (in_bom yes) (on_board yes)
-    (property "Reference" "U18" (id 0) (at 145.415 169.7798 0))
-    (property "Value" "LMV358MM" (id 1) (at 144.78 167.634 0)
-      (effects (font (size 1.27 1.27)) hide)
+    (property "Reference" "U18" (id 0) (at 147.32 167.8748 0))
+    (property "Value" "LMV358MM" (id 1) (at 147.32 169.539 0)
+      (effects (font (size 1.27 1.27) bold))
     )
     (property "Footprint" "Package_SO:SOIC-8_3.9x4.9mm_P1.27mm" (id 2) (at 143.51 173.99 0)
@@
     )
     (property "BMK-Nr" "11-0573" (id 4) (at 143.51 174.625 0)
-      (effects (font (size 1.27 1.27)) hide)
-    )
-    (property "Mouser" "926-LMV358MMX/NOPB" (id 4) (at 143.51 174.625 0)
       (effects (font (size 1.27 1.27)) hide)
     )
@@
   (symbol (lib_id "Kabeltester:74AHC2G08") (at 240.665 104.775 0) (unit 1)
     (in_bom yes) (on_board yes)
-    (property "Reference" "U22" (id 0) (at 240.665 97.155 0))
-    (property "Value" "74AHC2G08" (id 1) (at 241.3 95.885 0)
-      (effects (font (size 1.27 1.27)) hide)
+    (property "Reference" "U22" (id 0) (at 240.665 95.25 0))
+    (property "Value" "74AHC2G08" (id 1) (at 240.665 97.155 0)
+      (effects (font (size 1.27 1.27) bold))
     )
     (property "Footprint" "Package_SO:VSSOP-8_2.4x2.1mm_P0.5mm" (id 2) (at 252.73 116.205 0)
@@
   (symbol (lib_id "Kabeltester:74AHC2G08") (at 259.715 111.125 0) (unit 2)
     (in_bom yes) (on_board yes)
-    (property "Reference" "U22" (id 0) (at 259.715 103.505 0))
-    (property "Value" "74AHC2G08" (id 1) (at 260.35 102.235 0)
-      (effects (font (size 1.27 1.27)) hide)
+    (property "Reference" "U22" (id 0) (at 259.715 101.6 0))
+    (property "Value" "74AHC2G08" (id 1) (at 259.715 103.505 0)
+      (effects (font (size 1.27 1.27) bold))
     )
     (property "Footprint" "Package_SO:VSSOP-8_2.4x2.1mm_P0.5mm" (id 2) (at 271.78 122.555 0)
@@
   (symbol (lib_id "Kabeltester:INA826AIDRGT") (at 113.665 73.025 0) (mirror y) (unit 1)
     (in_bom yes) (on_board yes)
-    (property "Reference" "U19" (id 0) (at 110.49 64.8906 0))
-    (property "Value" "INA826AIDRGT" (id 1) (at 110.49 63.227 0)
-      (effects (font (size 1.27 1.27)) hide)
+    (property "Reference" "U19" (id 0) (at 119.38 61.7156 0))
+    (property "Value" "INA826AIDRGT" (id 1) (at 119.38 60.052 0)
+      (effects (font (size 1.27 1.27) bold))
     )
     (property "Footprint" "Package_DFN_QFN:DFN-8-1EP_2x2mm_P0.5mm_EP0.6x1.2mm" (id 2) (at 113.665 55.245 0)
@@
     )
     (property "BMK-Nr" "07-1477 / 07-2138" (id 4) (at 113.665 73.025 0)
-      (effects (font (size 1.27 1.27)) hide)
-    )
-    (property "Mouser" "595-INA826AIDGK" (id 4) (at 113.665 73.025 0)
       (effects (font (size 1.27 1.27)) hide)
     )
@@
   (symbol (lib_name "Kabeltester:74HC595_3") (lib_id "Kabeltester:74HC595") (at 346.71 118.745 0) (unit 1)
     (in_bom yes) (on_board yes)
-    (property "Reference" "U20" (id 0) (at 346.71 95.6118 0))
-    (property "Value" "74HC595" (id 1) (at 345.44 95.37 0)
-      (effects (font (size 1.27 1.27)) hide)
+    (property "Reference" "U20" (id 0) (at 346.71 94.3418 0))
+    (property "Value" "74HC595" (id 1) (at 346.71 96.005 0)
+      (effects (font (size 1.27 1.27) bold))
     )
     (property "Footprint" "Package_SO:TSSOP-16_4.4x5mm_P0.65mm" (id 2) (at 346.71 118.745 0)
@@
     )
     (property "BMK-Nr" "06-0831" (id 4) (at 346.71 118.745 0)
-      (effects (font (size 1.27 1.27)) hide)
-    )
-    (property "Mouser" "595-CD74HC595M96" (id 4) (at 346.71 118.745 0)
       (effects (font (size 1.27 1.27)) hide)
     )
@@
   (symbol (lib_id "Kabeltester:74HC595") (at 346.71 173.355 0) (unit 1)
     (in_bom yes) (on_board yes)
-    (property "Reference" "U21" (id 0) (at 346.71 150.2218 0))
-    (property "Value" "74HC595" (id 1) (at 342.265 173.475 90)
-      (effects (font (size 1.27 1.27)) hide)
+    (property "Reference" "U21" (id 0) (at 346.71 148.9518 0))
+    (property "Value" "74HC595" (id 1) (at 346.71 150.615 0)
+      (effects (font (size 1.27 1.27) bold))
     )
     (property "Footprint" "Package_SO:TSSOP-16_4.4x5mm_P0.65mm" (id 2) (at 346.71 173.355 0)
@@
       (effects (font (size 1.27 1.27)) hide)
     )
-    (property "Mouser" "595-CD74HC595M96" (id 4) (at 346.71 173.355 0)
-      (effects (font (size 1.27 1.27)) hide)
-    )
