File: 02_Schaltplan/KiCad/Schaltplan/Output.kicad_sch (KiCad schematic)
At the start: 22 parts, among them J10 Conn_02x01, J11 Conn_02x01, J12 Conn_02x01, J13 Conn_02x01, U23 74HC08PW

Commit message: ADD
-Dokumentation erweitert
-Schaltplan Fußbeschriftungen
Other:
- company: (none) -> BMK Group
- title: (none) -> Kabeltester
Changed lines of the file:
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@@
 (kicad_sch (version 20210126) (generator eeschema)
   (paper "A3")
+  (title_block
+    (title "Kabeltester")
+    (company "BMK Group")
+    (comment 1 "Erstellt: Maximilian Hoffmann")
+    (comment 2 "Geprüft: Robert Schulz")
+  )
   (junction (at 28.575 236.22) (diameter 1.016) (color 0 0 0 0))
   (junction (at 28.575 259.08) (diameter 1.016) (color 0 0 0 0))
