File: 02_Schaltplan/KiCad/Schaltplan/Kabeltester.kicad_sch (KiCad schematic)
At the start: 12 parts, among them J1 INPUT/MALE-DB9, J14 GND, J15 GND, J16 GND, J2 OUTPUT/FEMALE-DB9, J4 VCC

Commit message: ADD
-Dokumentation erweitert
-Schaltplan Fußbeschriftungen
Other:
- company: (none) -> BMK Group
- title: (none) -> Kabeltester
Changed lines of the file:
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@@
 (kicad_sch (version 20210126) (generator eeschema)
   (paper "A4")
+  (title_block
+    (title "Kabeltester")
+    (date "2021-04-12")
+    (company "BMK Group")
+    (comment 1 "Erstellt: Maximilian Hoffmann")
+    (comment 2 "Geprüft: Robert Schulz")
+  )
   (junction (at 47.625 177.165) (diameter 0.9144) (color 0 0 0 0))
   (junction (at 60.325 178.435) (diameter 0.9144) (color 0 0 0 0))
@@
     )
     (path "/19c6ec6d-ce00-421a-80b5-f5c992dce673/3cdba8fb-98a3-41b2-b01f-0d3910abb0f2"
-      (reference "D43") (unit 1) (value "D") (footprint "Diode_SMD:D_0805_2012Metric_Pad1.15x1.40mm_HandSolder")
+      (reference "D43") (unit 1) (value "BAS416") (footprint "Diode_SMD:D_0805_2012Metric_Pad1.15x1.40mm_HandSolder")
     )
     (path "/19c6ec6d-ce00-421a-80b5-f5c992dce673/19479609-6703-4575-a33f-ec8b8db026b7"
