File: 02_Schaltplan/KiCad/Schaltplan/Messumschaltung.kicad_sch (KiCad schematic)
At the start: 25 parts, among them U29 74HC86PW, U30 74HC02PW, U31 74HC02PW, U34 74HC08PW

Commit message: ADD
-Dokumentation erweitert
-Schaltplan Fußbeschriftungen
Other:
- company: (none) -> BMK Group
- title: (none) -> Kabeltester
Changed lines of the file:
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@@
 (kicad_sch (version 20210126) (generator eeschema)
   (paper "A3")
+  (title_block
+    (title "Kabeltester")
+    (company "BMK Group")
+    (comment 1 "Erstellt: Maximilian Hoffmann")
+    (comment 2 "Geprüft: Robert Schulz")
+  )
   (junction (at 23.495 231.14) (diameter 1.016) (color 0 0 0 0))
   (junction (at 23.495 251.46) (diameter 1.016) (color 0 0 0 0))

Commit message: Changes
Other:
- note removed: "DK-OUT-1 an Pin 4 anlöten"
- note removed: "Schutz vor extrem schnellen Nadelimpulse"
Changed lines of the file:
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@@
     (effects (font (size 3 3) (thickness 0.6) bold) (justify right bottom))
-  )
-  (text "Schutz vor extrem schnellen Nadelimpulse\n" (at 85.725 37.465 180)
-    (effects (font (size 1.27 1.27)) (justify right bottom))
-  )
-  (text "DK-OUT-1 an Pin 4 anlöten\n" (at 85.725 41.91 180)
-    (effects (font (size 1.27 1.27)) (justify right bottom))
   )
   (text "DK2\n" (at 103.505 51.435 180)
