File: 02_Schaltplan/KiCad/Schaltplan/Messumschaltung.kicad_sch (KiCad schematic)
At the start: 25 parts, among them U29 74HC86PW, U30 74HC02PW, U31 74HC02PW, U34 74HC08PW

Commit message: Änderungen
Connections:
- net SYSTEM_TACKT_SR renamed SYSTEM_TAKT_SR
- net SYSTEM_TACKT_SR_INV renamed SYSTEM_TAKT_SR_INV
- net SYSTEM_TACKT_SR_INV1 renamed SYSTEM_TAKT_SR_INV1
Changed lines of the file:
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@@
     )
   )
-  (global_label "SYSTEM_TACKT_SR_INV" (shape input) (at 36.83 22.225 180)
+  (global_label "SYSTEM_TAKT_SR_INV" (shape input) (at 36.83 22.225 180)
     (effects (font (size 1.27 1.27)) (justify right))
     (property "Intersheet References" "${INTERSHEET_REFS}" (id 0) (at 11.8472 22.3044 0)
@@
     )
   )
-  (global_label "SYSTEM_TACKT_SR_INV1" (shape input) (at 38.735 60.325 180)
+  (global_label "SYSTEM_TAKT_SR_INV1" (shape input) (at 38.735 60.325 180)
     (effects (font (size 1.27 1.27)) (justify right))
     (property "Intersheet References" "${INTERSHEET_REFS}" (id 0) (at 12.5427 60.2456 0)
@@
     )
   )
-  (global_label "SYSTEM_TACKT_SR_INV1" (shape input) (at 41.91 27.94 180)
+  (global_label "SYSTEM_TAKT_SR_INV1" (shape input) (at 41.91 27.94 180)
     (effects (font (size 1.27 1.27)) (justify right))
     (property "Intersheet References" "${INTERSHEET_REFS}" (id 0) (at 15.7177 27.8606 0)
@@
     )
   )
-  (global_label "SYSTEM_TACKT_SR" (shape input) (at 49.53 22.225 0)
+  (global_label "SYSTEM_TAKT_SR" (shape input) (at 49.53 22.225 0)
     (effects (font (size 1.27 1.27)) (justify left))
     (property "Intersheet References" "${INTERSHEET_REFS}" (id 0) (at 70.5214 22.1456 0)
@@
     )
   )
-  (global_label "SYSTEM_TACKT_SR_INV1" (shape input) (at 116.84 60.325 180)
+  (global_label "SYSTEM_TAKT_SR_INV1" (shape input) (at 116.84 60.325 180)
     (effects (font (size 1.27 1.27)) (justify right))
     (property "Intersheet References" "${INTERSHEET_REFS}" (id 0) (at 90.6477 60.2456 0)
@@
     )
   )
-  (global_label "SYSTEM_TACKT_SR_INV1" (shape input) (at 197.485 60.325 180)
+  (global_label "SYSTEM_TAKT_SR_INV1" (shape input) (at 197.485 60.325 180)
     (effects (font (size 1.27 1.27)) (justify right))
     (property "Intersheet References" "${INTERSHEET_REFS}" (id 0) (at 171.2927 60.2456 0)
@@
     )
   )
-  (global_label "SYSTEM_TACKT_SR_INV1" (shape input) (at 274.955 60.96 180)
+  (global_label "SYSTEM_TAKT_SR_INV1" (shape input) (at 274.955 60.96 180)
     (effects (font (size 1.27 1.27)) (justify right))
     (property "Intersheet References" "${INTERSHEET_REFS}" (id 0) (at 248.7627 60.8806 0)

Commit message: ADD
Connections:
- net SYSTEM_TAKT_SR: now also U34.10 (B), U34.12 (B), U34.2 (B), U34.5 (B)
- net SYSTEM_TAKT_SR_INV1: no longer U34.10 (B), U34.12 (B), U34.2 (B), U34.5 (B)
Other:
- moved on the sheet: C36, C37, C38, C39, C41, C42, C43, C47, R48, R49, R50, R51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

Commit message: ADD
Parts:
- U29: Stromaufnahme (none) -> 0.1uA
- U30, U31, U34: Stromaufnahme (none) -> 2uA
Changed lines of the file:
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@@
+      (effects (font (size 1.27 1.27)) hide)
+    )
+    (property "Stromaufnahme" "2uA" (id 4) (at 90.805 165.1 0)
       (effects (font (size 1.27 1.27)) hide)
     )
@@
       (effects (font (size 1.27 1.27)) hide)
     )
+    (property "Stromaufnahme" "0.1uA" (id 4) (at 28.575 165.1 0)
+      (effects (font (size 1.27 1.27)) hide)
+    )
     (pin "14")
     (pin "7")
@@
       (effects (font (size 1.27 1.27)) hide)
     )
+    (property "Stromaufnahme" "2uA" (id 4) (at 47.625 165.1 0)
+      (effects (font (size 1.27 1.27)) hide)
+    )
     (pin "14")
     (pin "7")
@@
       (effects (font (size 1.27 1.27)) hide)
     )
+    (property "Stromaufnahme" "2uA" (id 4) (at 67.31 165.1 0)
+      (effects (font (size 1.27 1.27)) hide)
+    )
     (pin "14")
     (pin "7")
@@
     )
     (property "Mouser" "771-HC08PW118" (id 5) (at 57.785 76.835 0)
+      (effects (font (size 1.27 1.27)) hide)
+    )
+    (property "Stromaufnahme" "2uA" (id 4) (at 49.53 57.15 0)
       (effects (font (size 1.27 1.27)) hide)
     )
@@
       (effects (font (size 1.27 1.27)) hide)
     )
+    (property "Stromaufnahme" "2uA" (id 4) (at 131.445 57.15 0)
+      (effects (font (size 1.27 1.27)) hide)
+    )
     (pin "4")
     (pin "5")
@@
       (effects (font (size 1.27 1.27)) hide)
     )
+    (property "Stromaufnahme" "2uA" (id 4) (at 214.63 114.935 0)
+      (effects (font (size 1.27 1.27)) hide)
+    )
     (pin "11")
     (pin "12")
@@
       (effects (font (size 1.27 1.27)) hide)
     )
+    (property "Stromaufnahme" "2uA" (id 4) (at 215.9 57.15 0)
+      (effects (font (size 1.27 1.27)) hide)
+    )
     (pin "10")
     (pin "8")
@@
       (effects (font (size 1.27 1.27)) hide)
     )
+    (property "Stromaufnahme" "0.1uA" (id 4) (at 49.53 79.375 0)
+      (effects (font (size 1.27 1.27)) hide)
+    )
     (pin "1")
     (pin "2")
@@
       (effects (font (size 1.27 1.27)) hide)
     )
+    (property "Stromaufnahme" "0.1uA" (id 4) (at 131.445 79.375 0)
+      (effects (font (size 1.27 1.27)) hide)
+    )
     (pin "4")
     (pin "5")
@@
       (effects (font (size 1.27 1.27)) hide)
     )
+    (property "Stromaufnahme" "0.1uA" (id 4) (at 214.63 137.16 0)
+      (effects (font (size 1.27 1.27)) hide)
+    )
     (pin "12")
     (pin "13")
@@
       (effects (font (size 1.27 1.27)) hide)
     )
+    (property "Stromaufnahme" "0.1uA" (id 4) (at 215.9 79.375 0)
+      (effects (font (size 1.27 1.27)) hide)
+    )
     (pin "9")
     (pin "10")
@@
       (effects (font (size 1.27 1.27)) hide)
     )
+    (property "Stromaufnahme" "2uA" (id 4) (at 71.755 57.15 0)
+      (effects (font (size 1.27 1.27)) hide)
+    )
     (pin "2")
     (pin "3")
@@
       (effects (font (size 1.27 1.27)) hide)
     )
+    (property "Stromaufnahme" "2uA" (id 4) (at 71.755 76.2 0)
+      (effects (font (size 1.27 1.27)) hide)
+    )
     (pin "5")
     (pin "6")
@@
       (effects (font (size 1.27 1.27)) hide)
     )
+    (property "Stromaufnahme" "2uA" (id 4) (at 153.67 57.15 0)
+      (effects (font (size 1.27 1.27)) hide)
+    )
     (pin "8")
     (pin "9")
@@
       (effects (font (size 1.27 1.27)) hide)
     )
+    (property "Stromaufnahme" "2uA" (id 4) (at 153.67 76.2 0)
+      (effects (font (size 1.27 1.27)) hide)
+    )
     (pin "11")
     (pin "12")
@@
       (effects (font (size 1.27 1.27)) hide)
     )
+    (property "Stromaufnahme" "2uA" (id 4) (at 236.855 114.935 0)
+      (effects (font (size 1.27 1.27)) hide)
+    )
     (pin "8")
     (pin "9")
@@
       (effects (font (size 1.27 1.27)) hide)
     )
+    (property "Stromaufnahme" "2uA" (id 4) (at 236.855 133.985 0)
+      (effects (font (size 1.27 1.27)) hide)
+    )
     (pin "11")
     (pin "12")
@@
       (effects (font (size 1.27 1.27)) hide)
     )
+    (property "Stromaufnahme" "2uA" (id 4) (at 238.125 57.15 0)
+      (effects (font (size 1.27 1.27)) hide)
+    )
     (pin "2")
     (pin "3")
@@
       (effects (font (size 1.27 1.27)) hide)
     )
+    (property "Stromaufnahme" "2uA" (id 4) (at 238.125 76.2 0)
+      (effects (font (size 1.27 1.27)) hide)
+    )

Commit message: Changes
Changed lines of the file:
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@@
     (effects (font (size 3 3) (thickness 0.6) bold) (justify right bottom))
   )
-  (text "Durchgangsprüfung &  Kurschlussmessung\n" (at 293.37 26.035 180)
+  (text "Durchgangsprüfung &  Kurschlussmessung\n" (at 241.935 26.67 180)
     (effects (font (size 5 5) (thickness 1) bold) (justify right bottom))
   )
@@
   (symbol (lib_id "Kabeltester:74HC08PW") (at 49.53 57.15 0) (unit 1)
     (in_bom yes) (on_board yes)
-    (property "Reference" "U34" (id 0) (at 49.53 49.53 0))
-    (property "Value" "74HC08PW" (id 1) (at 49.53 47.625 0)
-      (effects (font (size 1.27 1.27)) hide)
+    (property "Reference" "U34" (id 0) (at 49.53 47.625 0))
+    (property "Value" "74HC08PW" (id 1) (at 49.53 49.53 0)
+      (effects (font (size 1.27 1.27) bold))
     )
     (property "Footprint" "Package_SO:TSSOP-14_4.4x5mm_P0.65mm" (id 2) (at 55.88 72.39 0)
@@
   (symbol (lib_id "Kabeltester:74HC08PW") (at 131.445 57.15 0) (unit 2)
     (in_bom yes) (on_board yes)
-    (property "Reference" "U34" (id 0) (at 131.445 49.53 0))
-    (property "Value" "74HC08PW" (id 1) (at 131.445 47.625 0)
-      (effects (font (size 1.27 1.27)) hide)
+    (property "Reference" "U34" (id 0) (at 131.445 47.625 0))
+    (property "Value" "74HC08PW" (id 1) (at 131.445 49.53 0)
+      (effects (font (size 1.27 1.27) bold))
     )
     (property "Footprint" "Package_SO:TSSOP-14_4.4x5mm_P0.65mm" (id 2) (at 137.795 72.39 0)
@@
   (symbol (lib_id "Kabeltester:74HC08PW") (at 214.63 114.935 0) (unit 4)
     (in_bom yes) (on_board yes)
-    (property "Reference" "U34" (id 0) (at 214.63 107.315 0))
-    (property "Value" "74HC08PW" (id 1) (at 215.265 106.045 0)
-      (effects (font (size 1.27 1.27)) hide)
+    (property "Reference" "U34" (id 0) (at 214.63 105.41 0))
+    (property "Value" "74HC08PW" (id 1) (at 214.63 107.315 0)
+      (effects (font (size 1.27 1.27) bold))
     )
     (property "Footprint" "Package_SO:TSSOP-14_4.4x5mm_P0.65mm" (id 2) (at 220.98 130.175 0)
@@
   (symbol (lib_id "Kabeltester:74HC08PW") (at 215.9 57.15 0) (unit 3)
     (in_bom yes) (on_board yes)
-    (property "Reference" "U34" (id 0) (at 215.9 49.53 0))
-    (property "Value" "74HC08PW" (id 1) (at 215.9 47.625 0)
-      (effects (font (size 1.27 1.27)) hide)
+    (property "Reference" "U34" (id 0) (at 215.9 47.625 0))
+    (property "Value" "74HC08PW" (id 1) (at 215.9 49.53 0)
+      (effects (font (size 1.27 1.27) bold))
     )
     (property "Footprint" "Package_SO:TSSOP-14_4.4x5mm_P0.65mm" (id 2) (at 222.25 72.39 0)
@@
   (symbol (lib_id "Kabeltester:74HC86PW") (at 49.53 79.375 0) (unit 1)
     (in_bom yes) (on_board yes)
-    (property "Reference" "U29" (id 0) (at 49.53 71.755 0))
-    (property "Value" "74HC86PW" (id 1) (at 50.165 71.755 0)
-      (effects (font (size 1.27 1.27)) hide)
+    (property "Reference" "U29" (id 0) (at 49.53 88.9 0))
+    (property "Value" "74HC86PW" (id 1) (at 49.53 86.995 0)
+      (effects (font (size 1.27 1.27) bold))
     )
     (property "Footprint" "Package_SO:TSSOP-14_4.4x5mm_P0.65mm" (id 2) (at 49.53 104.775 0)
@@
   (symbol (lib_id "Kabeltester:74HC86PW") (at 131.445 79.375 0) (unit 2)
     (in_bom yes) (on_board yes)
-    (property "Reference" "U29" (id 0) (at 131.445 71.755 0))
-    (property "Value" "74HC86PW" (id 1) (at 132.08 71.12 0)
-      (effects (font (size 1.27 1.27)) hide)
+    (property "Reference" "U29" (id 0) (at 131.445 88.9 0))
+    (property "Value" "74HC86PW" (id 1) (at 131.445 86.995 0)
+      (effects (font (size 1.27 1.27) bold))
     )
     (property "Footprint" "Package_SO:TSSOP-14_4.4x5mm_P0.65mm" (id 2) (at 131.445 104.775 0)
@@
   (symbol (lib_id "Kabeltester:74HC86PW") (at 214.63 137.16 0) (unit 4)
     (in_bom yes) (on_board yes)
-    (property "Reference" "U29" (id 0) (at 214.63 129.54 0))
-    (property "Value" "74HC86PW" (id 1) (at 215.265 128.905 0)
-      (effects (font (size 1.27 1.27)) hide)
+    (property "Reference" "U29" (id 0) (at 214.63 146.685 0))
+    (property "Value" "74HC86PW" (id 1) (at 214.63 144.78 0)
+      (effects (font (size 1.27 1.27) bold))
     )
     (property "Footprint" "Package_SO:TSSOP-14_4.4x5mm_P0.65mm" (id 2) (at 214.63 162.56 0)
@@
   (symbol (lib_id "Kabeltester:74HC86PW") (at 215.9 79.375 0) (unit 3)
     (in_bom yes) (on_board yes)
-    (property "Reference" "U29" (id 0) (at 215.9 71.755 0))
-    (property "Value" "74HC86PW" (id 1) (at 215.9 71.755 0)
-      (effects (font (size 1.27 1.27)) hide)
+    (property "Reference" "U29" (id 0) (at 215.9 88.9 0))
+    (property "Value" "74HC86PW" (id 1) (at 215.9 86.995 0)
+      (effects (font (size 1.27 1.27) bold))
     )
     (property "Footprint" "Package_SO:TSSOP-14_4.4x5mm_P0.65mm" (id 2) (at 215.9 104.775 0)
@@
   (symbol (lib_name "Kabeltester:74HC02PW_1") (lib_id "Kabeltester:74HC02PW") (at 71.755 57.15 0) (unit 1)
     (in_bom yes) (on_board yes)
-    (property "Reference" "U30" (id 0) (at 71.755 49.53 0))
-    (property "Value" "74HC02PW" (id 1) (at 72.39 48.895 0)
-      (effects (font (size 1.27 1.27)) hide)
+    (property "Reference" "U30" (id 0) (at 71.755 47.625 0))
+    (property "Value" "74HC02PW" (id 1) (at 71.755 49.53 0)
+      (effects (font (size 1.27 1.27) bold))
     )
     (property "Footprint" "Package_SO:TSSOP-14_4.4x5mm_P0.65mm" (id 2) (at 74.295 81.915 0)
@@
   (symbol (lib_name "Kabeltester:74HC02PW_2") (lib_id "Kabeltester:74HC02PW") (at 71.755 76.2 0) (unit 2)
     (in_bom yes) (on_board yes)
-    (property "Reference" "U30" (id 0) (at 71.755 83.82 0))
-    (property "Value" "74HC02PW" (id 1) (at 73.025 68.58 0)
-      (effects (font (size 1.27 1.27)) hide)
+    (property "Reference" "U30" (id 0) (at 71.755 85.725 0))
+    (property "Value" "74HC02PW" (id 1) (at 74.295 83.82 0)
+      (effects (font (size 1.27 1.27) bold))
     )
     (property "Footprint" "Package_SO:TSSOP-14_4.4x5mm_P0.65mm" (id 2) (at 74.295 100.965 0)
@@
   (symbol (lib_id "Kabeltester:74HC02PW") (at 153.67 57.15 0) (unit 3)
     (in_bom yes) (on_board yes)
-    (property "Reference" "U30" (id 0) (at 153.67 49.53 0))
-    (property "Value" "74HC02PW" (id 1) (at 154.305 49.53 0)
-      (effects (font (size 1.27 1.27)) hide)
+    (property "Reference" "U30" (id 0) (at 153.67 47.625 0))
+    (property "Value" "74HC02PW" (id 1) (at 153.67 49.53 0)
+      (effects (font (size 1.27 1.27) bold))
     )
     (property "Footprint" "Package_SO:TSSOP-14_4.4x5mm_P0.65mm" (id 2) (at 156.21 81.915 0)
@@
   (symbol (lib_name "Kabeltester:74HC02PW_9") (lib_id "Kabeltester:74HC02PW") (at 153.67 76.2 0) (unit 4)
     (in_bom yes) (on_board yes)
-    (property "Reference" "U30" (id 0) (at 153.67 68.58 0))
-    (property "Value" "74HC02PW" (id 1) (at 154.305 68.58 0)
-      (effects (font (size 1.27 1.27)) hide)
+    (property "Reference" "U30" (id 0) (at 153.035 85.725 0))
+    (property "Value" "74HC02PW" (id 1) (at 155.575 83.82 0)
+      (effects (font (size 1.27 1.27) bold))
     )
     (property "Footprint" "Package_SO:TSSOP-14_4.4x5mm_P0.65mm" (id 2) (at 156.21 100.965 0)
@@
   (symbol (lib_name "Kabeltester:74HC02PW_7") (lib_id "Kabeltester:74HC02PW") (at 236.855 114.935 0) (unit 3)
     (in_bom yes) (on_board yes)
-    (property "Reference" "U31" (id 0) (at 236.855 107.315 0))
-    (property "Value" "74HC02PW" (id 1) (at 237.49 106.68 0)
-      (effects (font (size 1.27 1.27)) hide)
+    (property "Reference" "U31" (id 0) (at 236.855 105.41 0))
+    (property "Value" "74HC02PW" (id 1) (at 236.855 107.315 0)
+      (effects (font (size 1.27 1.27) bold))
     )
     (property "Footprint" "Package_SO:TSSOP-14_4.4x5mm_P0.65mm" (id 2) (at 239.395 139.7 0)
@@
   (symbol (lib_name "Kabeltester:74HC02PW_8") (lib_id "Kabeltester:74HC02PW") (at 236.855 133.985 0) (unit 4)
     (in_bom yes) (on_board yes)
-    (property "Reference" "U31" (id 0) (at 236.855 126.365 0))
-    (property "Value" "74HC02PW" (id 1) (at 237.49 125.73 0)
-      (effects (font (size 1.27 1.27)) hide)
+    (property "Reference" "U31" (id 0) (at 236.22 143.51 0))
+    (property "Value" "74HC02PW" (id 1) (at 238.76 141.605 0)
+      (effects (font (size 1.27 1.27) bold))
     )
     (property "Footprint" "Package_SO:TSSOP-14_4.4x5mm_P0.65mm" (id 2) (at 239.395 158.75 0)
@@
   (symbol (lib_name "Kabeltester:74HC02PW_5") (lib_id "Kabeltester:74HC02PW") (at 238.125 57.15 0) (unit 1)
     (in_bom yes) (on_board yes)
-    (property "Reference" "U31" (id 0) (at 238.125 49.53 0))
-    (property "Value" "74HC02PW" (id 1) (at 239.395 49.53 0)
-      (effects (font (size 1.27 1.27)) hide)
+    (property "Reference" "U31" (id 0) (at 238.125 47.625 0))
+    (property "Value" "74HC02PW" (id 1) (at 238.125 49.53 0)
+      (effects (font (size 1.27 1.27) bold))
     )
     (property "Footprint" "Package_SO:TSSOP-14_4.4x5mm_P0.65mm" (id 2) (at 240.665 81.915 0)
@@
   (symbol (lib_name "Kabeltester:74HC02PW_6") (lib_id "Kabeltester:74HC02PW") (at 238.125 76.2 0) (unit 2)
     (in_bom yes) (on_board yes)
-    (property "Reference" "U31" (id 0) (at 238.125 68.58 0))
-    (property "Value" "74HC02PW" (id 1) (at 238.76 68.58 0)
-      (effects (font (size 1.27 1.27)) hide)
+    (property "Reference" "U31" (id 0) (at 237.49 85.725 0))
+    (property "Value" "74HC02PW" (id 1) (at 240.03 83.82 0)
+      (effects (font (size 1.27 1.27) bold))
     )
     (property "Footprint" "Package_SO:TSSOP-14_4.4x5mm_P0.65mm" (id 2) (at 240.665 100.965 0)
