File: 02_Schaltplan/KiCad/Schaltplan/Versorgung.kicad_sch (KiCad schematic)
At the start: 31 parts, among them J5 9V_Batt, Q2 Si2301, SW3 PWR ON/OFF, U7 TPS_54331

Commit message: ADD
-Dokumentation erweitert
-Schaltplan Fußbeschriftungen
Other:
- company: (none) -> BMK Group
- title: (none) -> Kabeltester
Changed lines of the file:
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@@
 (kicad_sch (version 20210126) (generator eeschema)
   (paper "A4")
+  (title_block
+    (title "Kabeltester")
+    (company "BMK Group")
+    (comment 1 "Erstellt: Maximilian Hoffmann")
+    (comment 2 "Geprüft: Robert Schulz")
+  )
   (junction (at 44.45 95.25) (diameter 1.016) (color 0 0 0 0))
   (junction (at 53.975 146.05) (diameter 0.9144) (color 0 0 0 0))

Commit message: Changes
Other:
- note removed: "Überprüfe Footprint"
Changed lines of the file:
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@@
-    (effects (font (size 1.27 1.27) (thickness 0.254) bold) (justify right bottom))
-  )
-  (text "Überprüfe Footprint\n" (at 134.62 115.57 180)
     (effects (font (size 1.27 1.27) (thickness 0.254) bold) (justify right bottom))
   )
