File: 02_Schaltplan/KiCad/Schaltplan/Taktgeber.kicad_sch (KiCad schematic)
At the start: 43 parts, among them J3 SPEED (20k-POTI), SW2 MODE, U10 74AHC2G08, U11 NE555, U12 74AHC1G32, U13 74LVC1G175, U14 LTC6993, U15 74LVC1G175, U16 74LVC2G14, U8 74AHC1G14

Commit message: Inbetriebnahme 'Doc
Parts:
- J3: value SPEED (20k-POTI) -> 5k Poti
- R2: value 10k -> 12k
- R72: value 15k -> 10k
- R82: value 15k -> 2k
Other:
- note removed: "DIODE Fehlt"
Changed lines of the file:
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@@
     (effects (font (size 2 2) (thickness 0.4) bold) (justify right bottom))
-  )
-  (text "DIODE Fehlt\n" (at 41.275 48.26 180)
-    (effects (font (size 1.27 1.27) (thickness 0.254) bold) (justify right bottom))
   )
   (text "TAKT\n" (at 97.155 38.735 180)
@@
       (effects (font (size 1.27 1.27)) (justify left))
     )
-    (property "Value" "15k" (id 1) (at 22.098 83.064 90)
+    (property "Value" "2k" (id 1) (at 22.098 83.064 90)
       (effects (font (size 1.27 1.27)) (justify left))
     )
@@
       (effects (font (size 1.27 1.27)) (justify left))
     )
-    (property "Value" "10k" (id 1) (at 29.083 61.474 0)
+    (property "Value" "12k" (id 1) (at 29.083 61.474 0)
       (effects (font (size 1.27 1.27)) (justify left))
     )
@@
       (effects (font (size 1.27 1.27)) (justify left))
     )
-    (property "Value" "15k" (id 1) (at 30.353 72.269 0)
+    (property "Value" "10k" (id 1) (at 30.353 72.269 0)
       (effects (font (size 1.27 1.27)) (justify left))
     )
@@
     (in_bom yes) (on_board yes)
     (property "Reference" "J3" (id 0) (at 23.495 137.795 90))
-    (property "Value" "SPEED (20k-POTI)" (id 1) (at 31.115 142.875 90))
+    (property "Value" "5k Poti" (id 1) (at 31.115 142.875 90))
     (property "Footprint" "Potentiometer_THT:Potentiometer_ACP_CA6-H2,5_Horizontal" (id 2) (at 29.21 137.795 0)
       (effects (font (size 1.27 1.27)) hide)

Commit message: Doku
Schaltplan
-Versorgung
-Taktgeber
Parts:
- R2: value 12k -> 18k
- R72: value 10k -> 15k
- R82: value 2k -> NP
Connections:
- net SYSTEM_TACK: now also U8.2; no longer U8.4
- net at U13.3 (D): now also U8.4; no longer U8.2
Other:
- note removed: "Falsch herum"
- moved on the sheet: C10, C12, C13, C14, C15, C17, C18, C19, J3, U10C, U11B, U12B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

Commit message: Änderungen
Connections:
- net SYSTEM_TACK renamed SYSTEM_TAKT
- net SYSTEM_TACK_2 renamed SYSTEM_TAKT_2
Changed lines of the file:
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@@
     )
   )
-  (global_label "SYSTEM_TACK_2" (shape input) (at 194.31 63.5 0)
+  (global_label "SYSTEM_TAKT_2" (shape input) (at 194.31 63.5 0)
     (effects (font (size 1.27 1.27)) (justify left))
     (property "Intersheet References" "${INTERSHEET_REFS}" (id 0) (at 213.0638 63.4206 0)
@@
     )
   )
-  (global_label "SYSTEM_TACK_2" (shape input) (at 225.425 69.85 90)
+  (global_label "SYSTEM_TAKT_2" (shape input) (at 225.425 69.85 90)
     (effects (font (size 1.27 1.27)) (justify left))
     (property "Intersheet References" "${INTERSHEET_REFS}" (id 0) (at 225.3456 51.0962 90)
@@
     )
   )
-  (global_label "SYSTEM_TACK" (shape input) (at 264.16 76.2 0)
+  (global_label "SYSTEM_TAKT" (shape input) (at 264.16 76.2 0)
     (effects (font (size 1.27 1.27)) (justify left))
     (property "Intersheet References" "${INTERSHEET_REFS}" (id 0) (at 280.7366 76.1206 0)

Commit message: ADD
Other:
- note added: "TAKT TEILUNG"
- note added: "TAKT UMSCHALTUNG"
- note removed: "TAKT_TEILUNG"
- note removed: "TAKT_UMSCHALTUNG"
Changed lines of the file:
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@@
     (effects (font (size 2 2) (thickness 0.4) bold) (justify right bottom))
   )
-  (text "TAKT_UMSCHALTUNG\n" (at 143.51 38.735 180)
+  (text "TAKT UMSCHALTUNG\n" (at 143.51 38.735 180)
     (effects (font (size 2 2) (thickness 0.4) bold) (justify right bottom))
   )
@@
     (effects (font (size 5 5) (thickness 1) bold) (justify right bottom))
   )
-  (text "TAKT_TEILUNG\n\n" (at 248.285 42.545 180)
+  (text "TAKT TEILUNG\n\n" (at 248.285 42.545 180)
     (effects (font (size 2 2) (thickness 0.4) bold) (justify right bottom))
   )

Commit message: ADD
Other:
- note added: "Fehler 2"
Changed lines of the file:
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@@
     (stroke (width 1) (type solid) (color 0 0 255 1))
+  )
+  (polyline (pts (xy 241.935 44.45) (xy 241.935 54.61))
+    (stroke (width 0.3) (type dash_dot) (color 0 0 255 1))
+  )
+  (polyline (pts (xy 241.935 44.45) (xy 254.635 44.45))
+    (stroke (width 0.3) (type dash_dot) (color 0 0 255 1))
+  )
+  (polyline (pts (xy 254.635 44.45) (xy 254.635 54.61))
+    (stroke (width 0.3) (type dash_dot) (color 0 0 255 1))
+  )
+  (polyline (pts (xy 254.635 54.61) (xy 241.935 54.61))
+    (stroke (width 0.3) (type dash_dot) (color 0 0 255 1))
+  )
+  (polyline (pts (xy 256.54 47.625) (xy 256.54 45.085))
+    (stroke (width 0.3) (type solid) (color 0 0 255 1))
+  )
+  (polyline (pts (xy 256.54 47.625) (xy 259.08 48.26))
+    (stroke (width 0.3) (type solid) (color 0 0 255 1))
+  )
+  (polyline (pts (xy 256.54 47.625) (xy 262.255 43.18))
+    (stroke (width 0.3) (type solid) (color 0 0 255 1))
   )
   (polyline (pts (xy 279.4 31.75) (xy 279.4 120.65))
@@
     (effects (font (size 2 2) (thickness 0.4) bold) (justify right bottom))
   )
+  (text "Fehler 2\n" (at 270.51 43.18 180)
+    (effects (font (size 1.27 1.27) (thickness 0.254) bold) (justify right bottom))
+  )
   (global_label "NE55_OUT" (shape input) (at 86.995 76.2 0)

Commit message: ADD
Parts:
- D1, D2, D3, D4: Stromaufnahme (none) -> 1mA
- U10, U12, U8: Stromaufnahme (none) -> 1uA
- U11: Stromaufnahme (none) -> 2mA
- U13, U15, U16: Stromaufnahme (none) -> 0.1uA
- U14: Stromaufnahme (none) -> 65uA
Changed lines of the file:
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@@
+      (effects (font (size 1.27 1.27)) hide)
+    )
+    (property "Stromaufnahme" "1mA" (id 4) (at 139.7 53.975 0)
       (effects (font (size 1.27 1.27)) hide)
     )
@@
       (effects (font (size 1.27 1.27)) hide)
     )
+    (property "Stromaufnahme" "1mA" (id 4) (at 139.7 73.025 0)
+      (effects (font (size 1.27 1.27)) hide)
+    )
     (pin "1")
     (pin "2")
@@
       (effects (font (size 1.27 1.27)) hide)
     )
+    (property "Stromaufnahme" "1mA" (id 4) (at 225.425 99.06 0)
+      (effects (font (size 1.27 1.27)) hide)
+    )
     (pin "1")
     (pin "2")
@@
     )
     (property "Mouser" "604-APT1608LSYCKJ3RV" (id 4) (at 262.89 100.33 0)
+      (effects (font (size 1.27 1.27)) hide)
+    )
+    (property "Stromaufnahme" "1mA" (id 4) (at 262.89 100.33 0)
       (effects (font (size 1.27 1.27)) hide)
     )
@@
       (effects (font (size 1.27 1.27)) hide)
     )
+    (property "Stromaufnahme" "0.1uA" (id 4) (at 158.75 63.5 0)
+      (effects (font (size 1.27 1.27)) hide)
+    )
     (pin "6")
     (pin "1")
@@
       (effects (font (size 1.27 1.27)) hide)
     )
+    (property "Stromaufnahme" "0.1uA" (id 4) (at 194.31 133.35 0)
+      (effects (font (size 1.27 1.27)) hide)
+    )
     (pin "4")
     (pin "3")
@@
     )
     (property "Mouser" "771-74AHC1G14GW-G" (id 5) (at 235.585 19.685 0)
+      (effects (font (size 1.27 1.27)) hide)
+    )
+    (property "Stromaufnahme" "1uA" (id 4) (at 248.92 49.53 0)
       (effects (font (size 1.27 1.27)) hide)
     )
@@
       (effects (font (size 1.27 1.27)) hide)
     )
+    (property "Stromaufnahme" "1uA" (id 4) (at 28.575 171.45 0)
+      (effects (font (size 1.27 1.27)) hide)
+    )
     (pin "5")
     (pin "3")
@@
       (effects (font (size 1.27 1.27)) hide)
     )
+    (property "Stromaufnahme" "0.1uA" (id 4) (at 47.625 171.45 0)
+      (effects (font (size 1.27 1.27)) hide)
+    )
     (pin "5")
     (pin "2")
@@
       (effects (font (size 1.27 1.27)) hide)
     )
+    (property "Stromaufnahme" "1uA" (id 4) (at 66.675 171.45 0)
+      (effects (font (size 1.27 1.27)) hide)
+    )
     (pin "8")
     (pin "4")
@@
       (effects (font (size 1.27 1.27)) hide)
     )
+    (property "Stromaufnahme" "1uA" (id 4) (at 85.725 171.45 0)
+      (effects (font (size 1.27 1.27)) hide)
+    )
     (pin "5")
     (pin "3")
@@
     )
     (property "Mouser" "584-C6993CS6-2TRMPBF" (id 5) (at 160.02 200.66 0)
+      (effects (font (size 1.27 1.27)) hide)
+    )
+    (property "Stromaufnahme" "65uA" (id 4) (at 142.875 172.72 0)
       (effects (font (size 1.27 1.27)) hide)
     )
@@
       (effects (font (size 1.27 1.27)) hide)
     )
+    (property "Stromaufnahme" "0.1uA" (id 4) (at 123.825 171.45 0)
+      (effects (font (size 1.27 1.27)) hide)
+    )
     (pin "5")
     (pin "2")
@@
       (effects (font (size 1.27 1.27)) hide)
     )
+    (property "Stromaufnahme" "0.1uA" (id 4) (at 161.29 171.45 0)
+      (effects (font (size 1.27 1.27)) hide)
+    )
     (pin "5")
     (pin "2")
@@
     )
     (property "Mouser" "584-C6993CS6-2TRMPBF" (id 4) (at 104.775 171.45 0)
+      (effects (font (size 1.27 1.27)) hide)
+    )
+    (property "Stromaufnahme" "2mA" (id 5) (at 104.775 171.45 0)
       (effects (font (size 1.27 1.27)) hide)
     )
@@
     )
     (property "Mouser" "771-AHC2G08DC125" (id 5) (at 179.07 68.58 0)
+      (effects (font (size 1.27 1.27)) hide)
+    )
+    (property "Stromaufnahme" "1uA" (id 4) (at 168.275 50.8 0)
       (effects (font (size 1.27 1.27)) hide)
     )
@@
       (effects (font (size 1.27 1.27)) hide)
     )
+    (property "Stromaufnahme" "1uA" (id 4) (at 168.275 76.2 0)
+      (effects (font (size 1.27 1.27)) hide)
+    )
     (pin "1")
     (pin "2")
@@
       (effects (font (size 1.27 1.27)) hide)
     )
+    (property "Stromaufnahme" "1uA" (id 4) (at 187.325 63.5 0)
+      (effects (font (size 1.27 1.27)) hide)
+    )
     (pin "1")
     (pin "2")
@@
     )
     (property "Mouser" "771-74LVC1G175GW-G" (id 5) (at 202.565 141.605 0)
+      (effects (font (size 1.27 1.27)) hide)
+    )
+    (property "Stromaufnahme" "0.1uA" (id 4) (at 194.31 117.475 0)
       (effects (font (size 1.27 1.27)) hide)
     )
@@
       (effects (font (size 1.27 1.27)) hide)
     )
+    (property "Stromaufnahme" "0.1uA" (id 4) (at 248.92 76.2 0)
+      (effects (font (size 1.27 1.27)) hide)
+    )
     (pin "1")
     (pin "3")
@@
       (effects (font (size 1.27 1.27)) hide)
     )
+    (property "Stromaufnahme" "65uA" (id 4) (at 164.465 114.3 0)
+      (effects (font (size 1.27 1.27)) hide)
+    )
     (pin "6")
     (pin "1")
@@
       (effects (font (size 1.27 1.27)) hide)
     )
+    (property "Stromaufnahme" "2mA" (id 5) (at 67.31 76.2 0)
+      (effects (font (size 1.27 1.27)) hide)
+    )

Commit message: ddd
ADD's
Changes
Parts:
- R5, R7, R8: value 1k6 -> 3k3
- R6: value 1k2 -> 2k4
- U11: Mouser 584-C6993CS6-2TRMPBF -> (none)
Changed lines of the file:
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@@
       (effects (font (size 1.27 1.27)) (justify left))
     )
-    (property "Value" "1k6" (id 1) (at 150.616 51.943 90)
+    (property "Value" "3k3" (id 1) (at 150.616 51.943 90)
       (effects (font (size 1.27 1.27)) (justify left))
     )
@@
       (effects (font (size 1.27 1.27)) (justify left))
     )
-    (property "Value" "1k2" (id 1) (at 150.616 70.993 90)
+    (property "Value" "2k4" (id 1) (at 150.616 70.993 90)
       (effects (font (size 1.27 1.27)) (justify left))
     )
@@
       (effects (font (size 1.27 1.27)) (justify left))
     )
-    (property "Value" "1k6" (id 1) (at 226.568 86.239 0)
+    (property "Value" "3k3" (id 1) (at 226.568 86.239 0)
       (effects (font (size 1.27 1.27)) (justify left))
     )
@@
       (effects (font (size 1.27 1.27)) (justify left))
     )
-    (property "Value" "1k6" (id 1) (at 257.683 87.509 0)
+    (property "Value" "3k3" (id 1) (at 257.683 87.509 0)
       (effects (font (size 1.27 1.27)) (justify left))
     )
@@
       (effects (font (size 1.27 1.27)) hide)
     )
-    (property "Stromaufnahme" "1mA" (id 4) (at 139.7 53.975 0)
+    (property "Stromaufnahme" "1mA" (id 5) (at 139.7 53.975 0)
       (effects (font (size 1.27 1.27)) hide)
     )
@@
       (effects (font (size 1.27 1.27)) hide)
     )
-    (property "Stromaufnahme" "1mA" (id 4) (at 139.7 73.025 0)
+    (property "Stromaufnahme" "1mA" (id 5) (at 139.7 73.025 0)
       (effects (font (size 1.27 1.27)) hide)
     )
@@
       (effects (font (size 1.27 1.27)) hide)
     )
-    (property "Stromaufnahme" "1mA" (id 4) (at 225.425 99.06 0)
+    (property "Stromaufnahme" "1mA" (id 5) (at 225.425 99.06 0)
       (effects (font (size 1.27 1.27)) hide)
     )
@@
       (effects (font (size 1.27 1.27)) hide)
     )
-    (property "Stromaufnahme" "1mA" (id 4) (at 262.89 100.33 0)
+    (property "Stromaufnahme" "1mA" (id 5) (at 262.89 100.33 0)
       (effects (font (size 1.27 1.27)) hide)
     )
@@
       (effects (font (size 1.27 1.27)) hide)
     )
-    (property "Mouser" "584-C6993CS6-2TRMPBF" (id 4) (at 104.775 171.45 0)
-      (effects (font (size 1.27 1.27)) hide)
-    )
     (property "Stromaufnahme" "2mA" (id 5) (at 104.775 171.45 0)
       (effects (font (size 1.27 1.27)) hide)
@@
       (effects (font (size 1.27 1.27)) hide)
     )
-    (property "Mouser" "584-C6993CS6-2TRMPBF" (id 4) (at 67.31 76.2 0)
-      (effects (font (size 1.27 1.27)) hide)
-    )

Commit message: Changes
Parts:
- D1: Mouser 604-APT1608LSECKJ3RV -> (none)
- D2: Mouser 604-APT1608LZGCK -> (none)
- D3, D4: Mouser 604-APT1608LSYCKJ3RV -> (none)
Changed lines of the file:
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@@
     (stroke (width 1) (type solid) (color 0 0 255 1))
+  )
+  (text "TAKT\n" (at 27.94 37.465 180)
+    (effects (font (size 2 2) (thickness 0.4) bold) (justify right bottom))
   )
   (text "Versorgung" (at 37.465 151.13 180)
     (effects (font (size 2 2) (thickness 0.4) bold) (justify right bottom))
   )
-  (text "TAKT\n" (at 97.155 38.735 180)
-    (effects (font (size 2 2) (thickness 0.4) bold) (justify right bottom))
-  )
   (text "TAKT UMSCHALTUNG\n" (at 143.51 38.735 180)
     (effects (font (size 2 2) (thickness 0.4) bold) (justify right bottom))
@@
     (effects (font (size 5 5) (thickness 1) bold) (justify right bottom))
   )
-  (text "TAKT TEILUNG\n\n" (at 248.285 42.545 180)
+  (text "TAKT TEILUNG\n\n" (at 245.11 40.64 180)
     (effects (font (size 2 2) (thickness 0.4) bold) (justify right bottom))
   )
@@
   (symbol (lib_id "Connector:TestPoint") (at 260.985 76.2 0) (unit 1)
     (in_bom yes) (on_board yes)
-    (property "Reference" "TP28" (id 0) (at 259.08 70.485 0)
+    (property "Reference" "TP28" (id 0) (at 262.89 72.39 0)
       (effects (font (size 1.27 1.27)) (justify left))
     )
@@
       (effects (font (size 1.27 1.27)) hide)
     )
-    (property "Mouser" "604-APT1608LSECKJ3RV" (id 4) (at 139.7 53.975 0)
-      (effects (font (size 1.27 1.27)) hide)
-    )
     (property "Stromaufnahme" "1mA" (id 5) (at 139.7 53.975 0)
       (effects (font (size 1.27 1.27)) hide)
@@
       (effects (font (size 1.27 1.27)) hide)
     )
-    (property "Mouser" "604-APT1608LZGCK" (id 4) (at 139.7 73.025 0)
-      (effects (font (size 1.27 1.27)) hide)
-    )
     (property "Stromaufnahme" "1mA" (id 5) (at 139.7 73.025 0)
       (effects (font (size 1.27 1.27)) hide)
@@
       (effects (font (size 1.27 1.27)) hide)
     )
-    (property "Mouser" "604-APT1608LSYCKJ3RV" (id 4) (at 225.425 99.06 0)
-      (effects (font (size 1.27 1.27)) hide)
-    )
     (property "Stromaufnahme" "1mA" (id 5) (at 225.425 99.06 0)
       (effects (font (size 1.27 1.27)) hide)
@@
     )
     (property "BMK-Nr" "08-8619" (id 4) (at 262.89 100.33 0)
-      (effects (font (size 1.27 1.27)) hide)
-    )
-    (property "Mouser" "604-APT1608LSYCKJ3RV" (id 4) (at 262.89 100.33 0)
       (effects (font (size 1.27 1.27)) hide)
     )
@@
   (symbol (lib_id "Kabeltester:74LVC2G14") (at 158.75 63.5 90) (unit 1)
     (in_bom yes) (on_board yes)
-    (property "Reference" "U16" (id 0) (at 151.13 63.5 90)
+    (property "Reference" "U16" (id 0) (at 149.225 62.23 90)
       (effects (font (size 1.27 1.27)) (justify right))
     )
-    (property "Value" "74LVC2G14" (id 1) (at 163.83 64.77 90)
-      (effects (font (size 1.27 1.27)) (justify right) hide)
+    (property "Value" "74LVC2G14" (id 1) (at 145.415 64.135 90)
+      (effects (font (size 1.27 1.27) bold) (justify right))
     )
     (property "Footprint" "Package_TO_SOT_SMD:SOT-23-6_Handsoldering" (id 2) (at 187.325 62.865 0)
@@
   (symbol (lib_id "Kabeltester:74LVC2G14") (at 194.31 133.35 180) (unit 2)
     (in_bom yes) (on_board yes)
-    (property "Reference" "U16" (id 0) (at 194.31 129.54 0))
-    (property "Value" "74LVC2G14" (id 1) (at 194.31 127 0)
-      (effects (font (size 1.27 1.27)) hide)
+    (property "Reference" "U16" (id 0) (at 194.945 127 0))
+    (property "Value" "74LVC2G14" (id 1) (at 194.945 128.905 0)
+      (effects (font (size 1.27 1.27) bold))
     )
     (property "Footprint" "Package_TO_SOT_SMD:SOT-23-6_Handsoldering" (id 2) (at 193.675 104.775 0)
@@
   (symbol (lib_id "Kabeltester:74AHC1G14") (at 248.92 49.53 180) (unit 1)
     (in_bom yes) (on_board yes)
-    (property "Reference" "U8" (id 0) (at 247.015 46.355 0))
-    (property "Value" "74AHC1G14" (id 1) (at 247.65 55.245 0)
-      (effects (font (size 1.27 1.27)) hide)
+    (property "Reference" "U8" (id 0) (at 248.92 40.64 0))
+    (property "Value" "74AHC1G14" (id 1) (at 248.92 43.18 0)
+      (effects (font (size 1.27 1.27) bold))
     )
     (property "Footprint" "Package_TO_SOT_SMD:SOT-353_SC-70-5_Handsoldering" (id 2) (at 234.315 24.13 0)
@@
   (symbol (lib_name "Kabeltester:74AHC2G08_2") (lib_id "Kabeltester:74AHC2G08") (at 168.275 50.8 0) (unit 2)
     (in_bom yes) (on_board yes)
-    (property "Reference" "U10" (id 0) (at 168.275 43.18 0))
-    (property "Value" "74AHC2G08" (id 1) (at 169.545 41.91 0)
-      (effects (font (size 1.27 1.27)) hide)
+    (property "Reference" "U10" (id 0) (at 168.275 41.275 0))
+    (property "Value" "74AHC2G08" (id 1) (at 168.275 43.18 0)
+      (effects (font (size 1.27 1.27) bold))
     )
     (property "Footprint" "Package_SO:VSSOP-8_2.4x2.1mm_P0.5mm" (id 2) (at 167.64 34.29 0)
@@
   (symbol (lib_name "Kabeltester:74AHC2G08_1") (lib_id "Kabeltester:74AHC2G08") (at 168.275 76.2 0) (unit 1)
     (in_bom yes) (on_board yes)
-    (property "Reference" "U10" (id 0) (at 169.545 67.31 0))
-    (property "Value" "74AHC2G08" (id 1) (at 169.545 66.675 0)
-      (effects (font (size 1.27 1.27)) hide)
+    (property "Reference" "U10" (id 0) (at 168.275 66.675 0))
+    (property "Value" "74AHC2G08" (id 1) (at 168.275 68.58 0)
+      (effects (font (size 1.27 1.27) bold))
     )
     (property "Footprint" "Package_SO:VSSOP-8_2.4x2.1mm_P0.5mm" (id 2) (at 167.64 59.69 0)
@@
   (symbol (lib_name "Kabeltester:74AHC1G32_1") (lib_id "Kabeltester:74AHC1G32") (at 187.325 63.5 0) (unit 1)
     (in_bom yes) (on_board yes)
-    (property "Reference" "U12" (id 0) (at 188.595 54.61 0))
-    (property "Value" "74AHC1G32" (id 1) (at 187.96 53.975 0)
-      (effects (font (size 1.27 1.27)) hide)
+    (property "Reference" "U12" (id 0) (at 187.325 53.975 0))
+    (property "Value" "74AHC1G32" (id 1) (at 187.325 55.88 0)
+      (effects (font (size 1.27 1.27) bold))
     )
     (property "Footprint" "Package_TO_SOT_SMD:SOT-23-5_HandSoldering" (id 2) (at 187.325 63.5 0)
@@
   (symbol (lib_name "Kabeltester:74LVC1G175_2") (lib_id "Kabeltester:74LVC1G175") (at 194.31 117.475 0) (unit 1)
     (in_bom yes) (on_board yes)
-    (property "Reference" "U15" (id 0) (at 198.755 109.855 0))
-    (property "Value" "74LVC1G175" (id 1) (at 194.31 128.905 0)
-      (effects (font (size 1.27 1.27)) hide)
+    (property "Reference" "U15" (id 0) (at 200.66 107.95 0))
+    (property "Value" "74LVC1G175" (id 1) (at 201.295 109.855 0)
+      (effects (font (size 1.27 1.27) bold))
     )
     (property "Footprint" "Package_TO_SOT_SMD:SOT-363_SC-70-6_Handsoldering" (id 2) (at 187.325 108.585 0)
@@
   (symbol (lib_name "Kabeltester:74LVC1G175_3") (lib_id "Kabeltester:74LVC1G175") (at 248.92 76.2 0) (unit 1)
     (in_bom yes) (on_board yes)
-    (property "Reference" "U13" (id 0) (at 254 67.945 0))
-    (property "Value" "74LVC1G175" (id 1) (at 254 76.2 90)
-      (effects (font (size 1.27 1.27)) hide)
+    (property "Reference" "U13" (id 0) (at 255.905 66.04 0))
+    (property "Value" "74LVC1G175" (id 1) (at 255.905 68.58 0)
+      (effects (font (size 1.27 1.27) bold))
     )
     (property "Footprint" "Package_TO_SOT_SMD:SOT-363_SC-70-6_Handsoldering" (id 2) (at 241.935 67.31 0)
@@
   (symbol (lib_name "Kabeltester:LTC6993_1") (lib_id "Kabeltester:LTC6993") (at 164.465 114.3 0) (unit 1)
     (in_bom yes) (on_board yes)
-    (property "Reference" "U14" (id 0) (at 170.18 106.68 0))
-    (property "Value" "LTC6993" (id 1) (at 142.875 132.715 0)
-      (effects (font (size 1.27 1.27)) hide)
+    (property "Reference" "U14" (id 0) (at 171.45 104.775 0))
+    (property "Value" "LTC6993" (id 1) (at 170.18 106.68 0)
+      (effects (font (size 1.27 1.27) bold))
     )
     (property "Footprint" "Package_TO_SOT_SMD:SOT-23-6_Handsoldering" (id 2) (at 156.845 92.71 0)
@@
   (symbol (lib_id "Kabeltester:NE555") (at 67.31 76.2 0) (unit 1)
     (in_bom yes) (on_board yes)
-    (property "Reference" "U11" (id 0) (at 74.6761 58.5406 0)
-      (effects (font (size 1.27 1.27)) (justify left))
-    )
-    (property "Value" "NE555" (id 1) (at 62.611 79.254 90)
-      (effects (font (size 1.27 1.27)) (justify left) hide)
+    (property "Reference" "U11" (id 0) (at 75.3111 56.6356 0)
+      (effects (font (size 1.27 1.27)) (justify left))
+    )
+    (property "Value" "NE555" (id 1) (at 74.041 58.934 0)
+      (effects (font (size 1.27 1.27) bold) (justify left))
     )
     (property "Footprint" "Package_SO:SOIC-8_3.9x4.9mm_P1.27mm" (id 2) (at 104.775 43.18 0)
