File: 02_Schaltplan/KiCad/Schaltplan/Taktgeber.kicad_sch (KiCad schematic)
At the start: 43 parts, among them J3 5k Poti, SW2 MODE, U10 74AHC2G08, U11 NE555, U12 74AHC1G32, U13 74LVC1G175, U14 LTC6993, U15 74LVC1G175, U16 74LVC2G14, U8 74AHC1G14

Commit message: Changes
Parts:
- C9: value 3,9uF -> 4,7uF
Changed lines of the file:
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@@
       (effects (font (size 1.27 1.27)) (justify left))
     )
-    (property "Value" "3,9uF" (id 1) (at 38.481 102.114 0)
+    (property "Value" "4,7uF" (id 1) (at 38.481 102.114 0)
       (effects (font (size 1.27 1.27)) (justify left))
     )
