File: 02_Schaltplan/KiCad/Schaltplan/Kabeltester.kicad_pcb (KiCad board)
At the start: 4 copper layers, 99.7 x 99.7 mm, 253 parts, among them J1 INPUT/MALE-DB9, J10 Conn_02x01, J11 Conn_02x01, J12 Conn_02x01, J13 Conn_02x01, J14 GND, J15 GND, J16 GND, J2 OUTPUT/FEMALE-DB9, J3 SPEED (20k-POTI), J4 VCC, J5 9V_Batt, J6 MEASURE-CON, J7 MEASURE-CON, J8 MEASURE-CON, J9 MEASURE-CON, Q1 SI2318, Q10 Si2301, Q11 BC858, Q2 Si2301, Q3 BSS123, Q4 Si2301, Q5 BSS123, Q6 Si2301, Q7 BSS123, Q8 Si2301, Q9 BSS123, SW1 START, SW2 MODE, SW3 PWR ON/OFF, U1 74HC08PW, U10 74AHC2G08, U11 NE555, U12 74AHC1G32, U13 74LVC1G175, U14 LTC6993, U15 74LVC1G175, U16 74LVC2G14, U17 LMV321AUIDBVR, U18 LMV358MM, U19 INA826AIDRGT, U2 74HC02PW, U20 74HC595, U21 74HC595, U22 74AHC2G08, U23 74HC08PW, U28 74HC1G126, U29 74HC86PW, U3 74AHC1G32, U30 74HC02PW, U31 74HC02PW, U32 74AHC1G14, U34 74HC08PW, U38 DG2535, U39 DG2535, U4 74HC08PW, U5 CD74HC4514M96, U6 SN74LS93, U7 TPS_54331, U8 74AHC1G14

Commit message: ADD
Parts:
- added C26: 100nF, Capacitor_SMD:C_0603_1608Metric_Pad1.08x0.95mm_HandSolder, F.Cu at (297.9, 150.7)
- added R22: 10k, Resistor_SMD:R_0603_1608Metric_Pad0.98x0.95mm_HandSolder, F.Cu at (297.9, 153.2)
- added U9: 74AHC1G14, Package_TO_SOT_SMD:SOT-353_SC-70-5_Handsoldering, F.Cu at (292.8, 151.3)
- C22: value 10nF -> 1nF
- C51: value C -> 100nF
- D43: value D -> BAS416
- F1: value 500mA M -> 100mA M
- J3: value SPEED (20k-POTI) -> 5k Poti
- R11: value 1k -> 1k8
- R12: value 110R -> 1k
- R13: value 100mR -> 1R
- R2: value 10k -> 18k
- R43: value 100k -> 10k
- R73: value 681k -> 680k
- R74: value 137k -> 150k
- R82: value 15k -> NP
- R87, R88: value ? -> 1k
- R89: value ? -> 10k
- R90, R91: value ? -> 0R
- R92: value ? -> 22R
Connections:
- net Net-(C3-Pad2) renamed RST_DEZ
- net Net-(C32-Pad1) renamed +9V
- net Net-(TP22-Pad1) renamed OUT_RST_DEZ
- net Net-(U1-Pad5) renamed MEASURE_START
- R13 pad 1: Net-(L2-Pad1) -> Net-(R13-Pad1)
- R92 pad 2: Net-(L2-Pad1) -> Net-(R13-Pad1)
- U19 pad 1: Net-(L2-Pad1) -> Net-(R13-Pad1)
- U19 pad 7: Net-(C22-Pad1) -> Net-(R22-Pad1)
- U22 pad 2: SYSTEM_TACK_2 -> Net-(U22-Pad2)
- U8 pad 2: Net-(U13-Pad3) -> SYSTEM_TACK
- U8 pad 4: SYSTEM_TACK -> Net-(U13-Pad3)

Commit message: ADD
Parts:
- removed the C26 at (297.9, 150.7)
- removed R22: 10k, Resistor_SMD:R_0603_1608Metric_Pad0.98x0.95mm_HandSolder
- removed U9: 74AHC1G14, Package_TO_SOT_SMD:SOT-353_SC-70-5_Handsoldering
Changed lines of the file:
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@@
     )
   )
-  (footprint "Package_TO_SOT_SMD:SOT-353_SC-70-5_Handsoldering" (layer "F.Cu")
-    (at 292.7945 151.342)
-    (descr "SOT-353, SC-70-5, Handsoldering")
-    (tags "SOT-353 SC-70-5 Handsoldering")
-    (property "BMK-Nr" "06-0624")
-    (property "Mouser" "771-74AHC1G14GW-G")
-    (property "Sheetfile" "Constant-Current-Logic.kicad_sch")
-    (property "Sheetname" "Constant-Current-Logic")
-    (attr smd)
-    (fp_text reference "U9" (at 0 -2) (layer "F.SilkS")
-      (effects (font (size 1 1) (thickness 0.15)))
-    )
-    (fp_text value "74AHC1G14" (at 0 2 180) (layer "F.Fab")
-      (effects (font (size 1 1) (thickness 0.15)))
-    )
-    (fp_text user "${REFERENCE}" (at 0 0 90) (layer "F.Fab")
-      (effects (font (size 0.5 0.5) (thickness 0.075)))
-    )
-    (fp_line (start 0.7 -1.16) (end -1.2 -1.16) (layer "F.SilkS") (width 0.12))
-    (fp_line (start -0.7 1.16) (end 0.7 1.16) (layer "F.SilkS") (width 0.12))
-    (fp_line (start 2.4 1.4) (end 2.4 -1.4) (layer "F.CrtYd") (width 0.05))
-    (fp_line (start -2.4 1.4) (end 2.4 1.4) (layer "F.CrtYd") (width 0.05))
-    (fp_line (start -2.4 -1.4) (end 2.4 -1.4) (layer "F.CrtYd") (width 0.05))
-    (fp_line (start -2.4 -1.4) (end -2.4 1.4) (layer "F.CrtYd") (width 0.05))
-    (fp_line (start -0.175 -1.1) (end -0.675 -0.6) (layer "F.Fab") (width 0.1))
-    (fp_line (start 0.675 -1.1) (end -0.175 -1.1) (layer "F.Fab") (width 0.1))
-    (fp_line (start -0.675 -0.6) (end -0.675 1.1) (layer "F.Fab") (width 0.1))
-    (fp_line (start 0.675 -1.1) (end 0.675 1.1) (layer "F.Fab") (width 0.1))
-    (fp_line (start 0.675 1.1) (end -0.675 1.1) (layer "F.Fab") (width 0.1))
-    (pad "1" smd rect (at -1.33 -0.65) (locked) (size 1.5 0.4) (layers "F.Cu" "F.Paste" "F.Mask"))
-    (pad "2" smd rect (at -1.33 0) (locked) (size 1.5 0.4) (layers "F.Cu" "F.Paste" "F.Mask")
-      (net 26 "SYSTEM_TACK_2") (pintype "input"))
-    (pad "3" smd rect (at -1.33 0.65) (locked) (size 1.5 0.4) (layers "F.Cu" "F.Paste" "F.Mask")
-      (net 2 "GND") (pinfunction "GND") (pintype "bidirectional"))
-    (pad "4" smd rect (at 1.33 0.65) (locked) (size 1.5 0.4) (layers "F.Cu" "F.Paste" "F.Mask")
-      (net 196 "Net-(U22-Pad2)") (pintype "output"))
-    (pad "5" smd rect (at 1.33 -0.65) (locked) (size 1.5 0.4) (layers "F.Cu" "F.Paste" "F.Mask")
-      (net 6 "+5V") (pinfunction "VCC") (pintype "bidirectional"))
-    (model "${KICAD6_3DMODEL_DIR}/Package_TO_SOT_SMD.3dshapes/SOT-353_SC-70-5.wrl"
-      (offset (xyz 0 0 0))
-      (scale (xyz 1 1 1))
-      (rotate (xyz 0 0 0))
-    )
-  )
   (footprint "Resistor_SMD:R_0603_1608Metric_Pad0.98x0.95mm_HandSolder" (layer "F.Cu")
     (at 246.135 63.56 180)
@@
     )
   )
-  (footprint "Capacitor_SMD:C_0603_1608Metric_Pad1.08x0.95mm_HandSolder" (layer "F.Cu")
-    (at 297.8945 150.672)
-    (descr "Capacitor SMD 0603 (1608 Metric), square (rectangular) end terminal, IPC_7351 nominal with elongated pad for handsoldering. (Body size source: IPC-SM-782 page 76, https://www.pcb-3d.com/wordpress/wp-content/uploads/ipc-sm-782a_amendment_1_and_2.pdf), generated with kicad-footprint-generator")
-    (tags "capacitor handsolder")
-    (property "BMK-Nr" "BS")
-    (property "Sheetfile" "Constant-Current-Logic.kicad_sch")
-    (property "Sheetname" "Constant-Current-Logic")
-    (attr smd)
-    (fp_text reference "C26" (at 0 -1.43) (layer "F.SilkS")
-      (effects (font (size 1 1) (thickness 0.15)))
-    )
-    (fp_text value "100nF" (at 0 1.43) (layer "F.Fab")
-      (effects (font (size 1 1) (thickness 0.15)))
-    )
-    (fp_text user "${REFERENCE}" (at 0 0) (layer "F.Fab")
-      (effects (font (size 0.4 0.4) (thickness 0.06)))
-    )
-    (fp_line (start -0.146267 -0.51) (end 0.146267 -0.51) (layer "F.SilkS") (width 0.12))
-    (fp_line (start -0.146267 0.51) (end 0.146267 0.51) (layer "F.SilkS") (width 0.12))
-    (fp_line (start -1.65 -0.73) (end 1.65 -0.73) (layer "F.CrtYd") (width 0.05))
-    (fp_line (start 1.65 0.73) (end -1.65 0.73) (layer "F.CrtYd") (width 0.05))
-    (fp_line (start -1.65 0.73) (end -1.65 -0.73) (layer "F.CrtYd") (width 0.05))
-    (fp_line (start 1.65 -0.73) (end 1.65 0.73) (layer "F.CrtYd") (width 0.05))
-    (fp_line (start -0.8 -0.4) (end 0.8 -0.4) (layer "F.Fab") (width 0.1))
-    (fp_line (start 0.8 -0.4) (end 0.8 0.4) (layer "F.Fab") (width 0.1))
-    (fp_line (start -0.8 0.4) (end -0.8 -0.4) (layer "F.Fab") (width 0.1))
-    (fp_line (start 0.8 0.4) (end -0.8 0.4) (layer "F.Fab") (width 0.1))
-    (pad "1" smd roundrect (at -0.8625 0) (locked) (size 1.075 0.95) (layers "F.Cu" "F.Paste" "F.Mask") (roundrect_rratio 0.25)
-      (net 6 "+5V") (pintype "passive"))
-    (pad "2" smd roundrect (at 0.8625 0) (locked) (size 1.075 0.95) (layers "F.Cu" "F.Paste" "F.Mask") (roundrect_rratio 0.25)
-      (net 2 "GND") (pintype "passive"))
-    (model "${KICAD6_3DMODEL_DIR}/Capacitor_SMD.3dshapes/C_0603_1608Metric.wrl"
-      (offset (xyz 0 0 0))
-      (scale (xyz 1 1 1))
-      (rotate (xyz 0 0 0))
-    )
-  )
   (footprint "Package_SO:TSSOP-14_4.4x5mm_P0.65mm" (layer "F.Cu")
     (at 206.13 134.9575 -90)
@@
       (offset (xyz 0 0 0))
       (scale (xyz 1 1 1))
-      (rotate (xyz 0 0 0))
-    )
-  )
-  (footprint "Resistor_SMD:R_0603_1608Metric_Pad0.98x0.95mm_HandSolder" (layer "F.Cu")
-    (at 297.8945 153.182)
-    (descr "Resistor SMD 0603 (1608 Metric), square (rectangular) end terminal, IPC_7351 nominal with elongated pad for handsoldering. (Body size source: IPC-SM-782 page 72, https://www.pcb-3d.com/wordpress/wp-content/uploads/ipc-sm-782a_amendment_1_and_2.pdf), generated with kicad-footprint-generator")
-    (tags "resistor handsolder")
-    (property "BMK-Nr" "BS")
-    (property "Mouser" "-")
-    (property "Sheetfile" "Constant-Current-Logic.kicad_sch")
-    (property "Sheetname" "Constant-Current-Logic")
-    (attr smd)
-    (fp_text reference "R22" (at 0 -1.43) (layer "F.SilkS")
-      (effects (font (size 0.5 0.5) (thickness 0.1)))
-    )
-    (fp_text value "10k" (at 0 1.43) (layer "F.Fab")
-      (effects (font (size 1 1) (thickness 0.15)))
-    )
-    (fp_text user "${REFERENCE}" (at 0 0) (layer "F.Fab")
-      (effects (font (size 0.4 0.4) (thickness 0.06)))
-    )
-    (fp_line (start -0.254724 -0.5225) (end 0.254724 -0.5225) (layer "F.SilkS") (width 0.12))
-    (fp_line (start -0.254724 0.5225) (end 0.254724 0.5225) (layer "F.SilkS") (width 0.12))
-    (fp_line (start 1.65 -0.73) (end 1.65 0.73) (layer "F.CrtYd") (width 0.05))
-    (fp_line (start -1.65 0.73) (end -1.65 -0.73) (layer "F.CrtYd") (width 0.05))
-    (fp_line (start -1.65 -0.73) (end 1.65 -0.73) (layer "F.CrtYd") (width 0.05))
-    (fp_line (start 1.65 0.73) (end -1.65 0.73) (layer "F.CrtYd") (width 0.05))
-    (fp_line (start 0.8 -0.4125) (end 0.8 0.4125) (layer "F.Fab") (width 0.1))
-    (fp_line (start 0.8 0.4125) (end -0.8 0.4125) (layer "F.Fab") (width 0.1))
-    (fp_line (start -0.8 0.4125) (end -0.8 -0.4125) (layer "F.Fab") (width 0.1))
-    (fp_line (start -0.8 -0.4125) (end 0.8 -0.4125) (layer "F.Fab") (width 0.1))
-    (pad "1" smd roundrect (at -0.9125 0) (locked) (size 0.975 0.95) (layers "F.Cu" "F.Paste" "F.Mask") (roundrect_rratio 0.25)
-      (net 168 "Net-(R22-Pad1)") (pintype "passive"))
-    (pad "2" smd roundrect (at 0.9125 0) (locked) (size 0.975 0.95) (layers "F.Cu" "F.Paste" "F.Mask") (roundrect_rratio 0.25)
-      (net 25 "Net-(C22-Pad1)") (pintype "passive"))
-    (model "${KICAD6_3DMODEL_DIR}/Resistor_SMD.3dshapes/R_0603_1608Metric.wrl"
-      (offset (xyz 0 0 0))
-      (scale (xyz 1 1 1))
