File: 02_Schaltplan/KiCad/Bestückungsplan/Constant-Current-Logic.kicad_sch (KiCad schematic)
At the start: 42 parts, among them Q1 SI2318, U17 LMV321AUIDBVR, U18 LMV358MM, U19 INA826AIDRGT, U20 74HC595, U21 74HC595, U22 74AHC2G08

Commit message: Changes & ADD
+Bestückungsplan
+Auftragsplannung
@ Klärung verschiedener Begrifflichkeiten
Other:
- note removed: "Hysterese-Widerstand"
Changed lines of the file:
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@@
     (effects (font (size 1.27 1.27) (thickness 0.254) bold) (justify right bottom))
-  )
-  (text "Hysterese-Widerstand\n" (at 178.435 168.275 180)
-    (effects (font (size 1.27 1.27)) (justify right bottom))
   )
   (text "LVC-Variante nehmen \nist bei BMK vorrätig\n\n1* 4AND\n1 * 2NOT\n\n"
