File: 02_Schaltplan/KiCad/Schaltplan_V001/Taktgeber.kicad_sch (KiCad schematic)
At the start: 43 parts, among them J3 SPEED (20k-POTI), SW2 MODE, U10 74AHC2G08, U11 NE555, U12 74AHC1G32, U13 74LVC1G175, U14 LTC6993, U15 74LVC1G175, U16 74LVC2G14, U8 74AHC1G14

Commit message: ADD & Changes
Inbetriebnahme Tex
Other:
- note removed: "Falsch herum"
Changed lines of the file:
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@@
     (effects (font (size 2 2) (thickness 0.4) bold) (justify right bottom))
-  )
-  (text "Falsch herum\n" (at 264.795 45.72 180)
-    (effects (font (size 1.27 1.27)) (justify right bottom))
   )
   (global_label "NE55_OUT" (shape input) (at 86.995 76.2 0)
