File: 02_Schaltplan/KiCad/Schaltplan_Prototype/Versorgung.kicad_sch (KiCad schematic)
At the start: 31 parts, among them J5 9V_Batt, Q2 Si2301, SW3 PWR ON/OFF, U7 TPS_54331

Commit message: ADD
Other:
- note added: "Fehler 1"
- note removed: "Passende Wago-Klemme suchen"
Changed lines of the file:
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@@
     (stroke (width 1) (type solid) (color 0 0 255 1))
+  )
+  (polyline (pts (xy 50.165 97.79) (xy 51.435 97.155))
+    (stroke (width 0.3) (type solid) (color 0 0 255 1))
+  )
+  (polyline (pts (xy 51.435 97.155) (xy 50.165 100.965))
+    (stroke (width 0.3) (type solid) (color 0 0 255 1))
+  )
+  (polyline (pts (xy 51.435 97.155) (xy 52.07 98.425))
+    (stroke (width 0.3) (type solid) (color 0 0 255 1))
   )
   (polyline (pts (xy 57.15 31.75) (xy 25.4 31.75))
@@
     (stroke (width 1) (type solid) (color 0 0 255 1))
   )
-  (text "Passende Wago-Klemme suchen\n" (at 57.785 29.845 180)
-    (effects (font (size 1.27 1.27) (thickness 0.254) bold) (justify right bottom))
+  (text "Fehler 1" (at 55.88 104.14 180)
+    (effects (font (size 1.5 1.5) (thickness 0.3) bold) (justify right bottom))
   )
   (text "VERSORGUNG\n" (at 177.8 33.655 180)
