File: 02_Schaltplan/KiCad/Schaltplan_Prototype/_autosave-Constant-Current-Logic.kicad_sch (KiCad schematic)
At the start: 40 parts, among them Q1 SI2318, U17 LMV321AUIDBVR, U18 LMV358MM, U19 INA826AIDRGT, U20 74HC595, U21 74HC595, U22 74AHC2G08

Commit message: ADD
Parts:
- R92: value 0R -> 22R
- U20, U21: footprint Package_SO:TSSOP-16_4.4x5mm_P0.65mm -> Package_SO:SOIC-16_3.9x9.9mm_P1.27mm; BMK-Nr 06-0831 -> 06-0163
Other:
- note added: "Fehler 3"
- note added: "Fehler 4"
- note added: "Fehler 5"
- note added: "Konstantstrom-Logik"
- note removed: "CONSTANT-CURRENT-LOGIC"
- moved on the sheet: JP1, JP2, TP36, TP37, TP6, TP7, U22A, U22B
