File: 02_Schaltplan/KiCad/Schaltplan_Prototype/_autosave-Taktgeber.kicad_sch (KiCad schematic)
At the start: 43 parts, among them J3 SPEED (20k-POTI), SW2 MODE, U10 74AHC2G08, U11 NE555, U12 74AHC1G32, U13 74LVC1G175, U14 LTC6993, U15 74LVC1G175, U16 74LVC2G14, U8 74AHC1G14

Commit message: ADD
Other:
- note added: "Fehler 2"
- note removed: "DIODE Fehlt"
Changed lines of the file:
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@@
     (stroke (width 1) (type solid) (color 0 0 255 1))
+  )
+  (polyline (pts (xy 253.365 44.45) (xy 252.73 43.18))
+    (stroke (width 0.3) (type solid) (color 0 0 255 1))
+  )
+  (polyline (pts (xy 253.365 44.45) (xy 254.635 41.275))
+    (stroke (width 0.3) (type solid) (color 0 0 255 1))
+  )
+  (polyline (pts (xy 254.635 43.815) (xy 253.365 44.45))
+    (stroke (width 0.3) (type solid) (color 0 0 255 1))
   )
   (polyline (pts (xy 279.4 31.75) (xy 279.4 120.65))
@@
   (text "Versorgung" (at 37.465 157.48 180)
     (effects (font (size 2 2) (thickness 0.4) bold) (justify right bottom))
-  )
-  (text "DIODE Fehlt\n" (at 41.275 48.26 180)
-    (effects (font (size 1.27 1.27) (thickness 0.254) bold) (justify right bottom))
   )
   (text "TAKT\n" (at 97.155 38.735 180)
@@
     (effects (font (size 2 2) (thickness 0.4) bold) (justify right bottom))
   )
+  (text "Fehler 2" (at 262.255 41.275 180)
+    (effects (font (size 1.5 1.5) (thickness 0.3) bold) (justify right bottom))
+  )
   (global_label "NE55_OUT" (shape input) (at 86.995 76.2 0)
