File: 02_Schaltplan/KiCad/Schaltplan_Prototype/Constant-Current-Logic.kicad_sch (KiCad schematic)
At the start: 40 parts, among them Q1 SI2318, U17 LMV321AUIDBVR, U18 LMV358MM, U19 INA826AIDRGT, U20 74HC595, U21 74HC595, U22 74AHC2G08

Commit message: Doku
Schaltplan
-Versorgung
-Taktgeber
Parts:
- U20, U21: footprint Package_SO:TSSOP-16_4.4x5mm_P0.65mm -> Package_SO:SOIC-16_3.9x9.9mm_P1.27mm; BMK-Nr 06-0831 -> 06-0163
Other:
- note added: "Konstantstrom-Logik"
- note removed: "CONSTANT-CURRENT-LOGIC"
Changed lines of the file:
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@@
     (effects (font (size 1.5 1.5) (thickness 0.3) bold) (justify right bottom))
   )
-  (text "CONSTANT-CURRENT-LOGIC\n" (at 274.955 27.305 180)
+  (text "Konstantstrom-Logik\n\n" (at 267.97 41.275 180)
     (effects (font (size 5 5) (thickness 1) bold) (justify right bottom))
   )
@@
       (effects (font (size 1.27 1.27)) hide)
     )
-    (property "Footprint" "Package_SO:TSSOP-16_4.4x5mm_P0.65mm" (id 2) (at 363.22 115.57 0)
+    (property "Footprint" "Package_SO:SOIC-16_3.9x9.9mm_P1.27mm" (id 2) (at 363.22 115.57 0)
       (effects (font (size 1.27 1.27)) hide)
     )
@@
       (effects (font (size 1.27 1.27)) hide)
     )
-    (property "BMK-Nr" "06-0831" (id 4) (at 363.22 115.57 0)
+    (property "BMK-Nr" "06-0163" (id 4) (at 363.22 115.57 0)
       (effects (font (size 1.27 1.27)) hide)
     )
@@
       (effects (font (size 1.27 1.27)) hide)
     )
-    (property "Footprint" "Package_SO:TSSOP-16_4.4x5mm_P0.65mm" (id 2) (at 363.22 170.18 0)
+    (property "Footprint" "Package_SO:SOIC-16_3.9x9.9mm_P1.27mm" (id 2) (at 363.22 170.18 0)
       (effects (font (size 1.27 1.27)) hide)
     )
@@
       (effects (font (size 1.27 1.27)) hide)
     )
-    (property "BMK-Nr" "06-0831" (id 4) (at 363.22 170.18 0)
-      (effects (font (size 1.27 1.27)) hide)
-    )
+    (property "BMK-Nr" "06-0163" (id 4) (at 363.22 170.18 0)
+      (effects (font (size 1.27 1.27)) hide)
+    )
