File: 02_Schaltplan/KiCad/Schaltplan_Prototype/Kabeltester.kicad_sch (KiCad schematic)
At the start: 12 parts, among them J1 INPUT/MALE-DB9, J14 GND, J15 GND, J16 GND, J2 OUTPUT/FEMALE-DB9, J4 VCC

Commit message: Doku
Schaltplan
-Versorgung
-Taktgeber
Other:
- note added: "Abschlussprojekt Kabeltester Prototyp V-01"
- note removed: "Abschlussprojekt Kabeltester Prototype V-01"
Changed lines of the file:
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@@
     (stroke (width 1) (type solid) (color 0 255 0 1))
   )
-  (text "Abschlussprojekt\nKabeltester\nPrototype V-01\n" (at 177.8 43.18 180)
+  (text "Abschlussprojekt\nKabeltester\nPrototyp V-01\n" (at 177.8 43.18 180)
     (effects (font (size 5 5) (thickness 1) bold) (justify right bottom))
   )
@@
     )
     (path "/9dfedc54-4d5e-45ef-a50a-32628d446e72/9b7f76d9-69f6-4452-ba17-132edaf9927d"
-      (reference "U20") (unit 1) (value "74HC595") (footprint "Package_SO:TSSOP-16_4.4x5mm_P0.65mm")
+      (reference "U20") (unit 1) (value "74HC595") (footprint "Package_SO:SOIC-16_3.9x9.9mm_P1.27mm")
     )
     (path "/9dfedc54-4d5e-45ef-a50a-32628d446e72/a92ede32-c6e2-44a7-bfda-6ec7fae74b9a"
@@
     )
     (path "/9dfedc54-4d5e-45ef-a50a-32628d446e72/3c8d2cb5-7abf-4720-af24-5134a4acc7b7"
-      (reference "U21") (unit 1) (value "74HC595") (footprint "Package_SO:TSSOP-16_4.4x5mm_P0.65mm")
+      (reference "U21") (unit 1) (value "74HC595") (footprint "Package_SO:SOIC-16_3.9x9.9mm_P1.27mm")
     )
     (path "/9dfedc54-4d5e-45ef-a50a-32628d446e72/c89a7242-604e-4ac2-9d9c-39d6f138c285"
