File: 02_Schaltplan/KiCad/Schaltplan_Prototype/Taktgeber.kicad_sch (KiCad schematic)
At the start: 43 parts, among them J3 SPEED (20k-POTI), SW2 MODE, U10 74AHC2G08, U11 NE555, U12 74AHC1G32, U13 74LVC1G175, U14 LTC6993, U15 74LVC1G175, U16 74LVC2G14, U8 74AHC1G14

Commit message: Doku
Schaltplan
-Versorgung
-Taktgeber
Other:
- note removed: "DIODE Fehlt"
Changed lines of the file:
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@@
     (effects (font (size 2 2) (thickness 0.4) bold) (justify right bottom))
-  )
-  (text "DIODE Fehlt\n" (at 41.275 48.26 180)
-    (effects (font (size 1.27 1.27) (thickness 0.254) bold) (justify right bottom))
   )
   (text "TAKT\n" (at 97.155 38.735 180)
